File: Hardware/ESPSoM/ESPSoM_HW00/ESPSoM_HW00/Connectors.kicad_sch (KiCad schematic)
At the start: 4 parts, among them J101 USB4510-03-1-A

Commit message: schematic first commit
Parts:
- removed BT101: Battery_Cell, Component_lib:BatteryHolder_Keystone_1042_1x18650_DUALSIDE, symbol Device:Battery_Cell
- added J1: 54722-0604, 547220604, symbol Component_lib:54722-0604
Connections:
- net D+: now also J1.58
- net D-: now also J1.57
- net GND: now also J1.1, J1.11, J1.12, J1.2, J1.55, J1.56, J1.59, J1.60
- net VBAT: now also J1.7, J1.9
- net VBUS: now also J1.3, J1.5
- new net +3V3: J1.4, J1.6
- new net IO0: J1.14
- new net IO1: J1.16
- new net IO10: J1.34
- new net IO11: J1.36
- new net IO12: J1.38
- new net IO13: J1.40
- new net IO14: J1.42
- new net IO15: J1.44
- new net IO16: J1.46
- new net IO17: J1.48
- new net IO18: J1.50
- new net IO2: J1.18
- new net IO21: J1.52
- new net IO3: J1.20
- new net IO33: J1.54
- new net IO34: J1.37
- new net IO35: J1.39
- new net IO36: J1.41
- new net IO37: J1.43
- new net IO38: J1.45
- new net IO39: J1.47
- new net IO4: J1.22
- new net IO40: J1.49
- new net IO41: J1.51
- new net IO42: J1.53
- new net IO5: J1.24
- new net IO6: J1.26
- new net IO7: J1.28
- new net IO8: J1.30
- new net IO9: J1.32
- new net VSYS: J1.10, J1.8
