File: Hardware/ESPSoM/ESPSoM_HW00/ESPSoM_HW00/ESP32S2FH4S2.kicad_sch (KiCad schematic)
At the start: 33 parts, among them J401 Conn_01x08_Female, J402 Conn_01x03_Socket, U401 ESP32-S2FH4, Y601 Crystal_GND24_Small

Commit message: schematic first commit
Parts:
- removed J401: Conn_01x08_Female, Connector_PinHeader_1.27mm:PinHeader_1x08_P1.27mm_Vertical, symbol Connector:Conn_01x08_Female
- removed J402: Conn_01x03_Socket, Connector_PinHeader_2.54mm:PinHeader_1x03_P2.54mm_Vertical, symbol Connector:Conn_01x03_Socket
Connections:
- net IO15: now also U401.21 (XTAL_32K_P)
- net BTN renamed IO14
- net DOWN renamed IO11
- net LED renamed IO9
- net LED_EN renamed IO21
- net LED_MOSI renamed IO39
- net LEFT renamed IO12
- net PL renamed IO7
- net RIGHT renamed IO13
- net SR_CLK renamed IO6
- net SR_CS renamed IO5
- net SR_MISO renamed IO8
- net UP renamed IO10
