File: Hardware/ESPSoM/ESPSoM_HW00/ESPSoM_HW00/ESPSoM_HW00.kicad_sch (KiCad schematic)
At the start: 1 part, among them J1 54722-0604

Commit message: schematic first commit
Parts:
- removed J1: 54722-0604, 547220604, symbol Component_lib:54722-0604
Other:
- sheet 1S_Charger renamed 200_1S_Charger
- added sheet 100_Connectors (Connectors.kicad_sch)
- added sheet 300_Power (Power.kicad_sch)
- added sheet 400_ESP32 (ESP32S2FH4S2.kicad_sch)
- sheet 200_1S_Charger ports: added GND, VBAT, VBUS, VSYS; removed none
Changed lines of the file:
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@@
 (kicad_sch (version 20230121) (generator eeschema)
   (paper "A4")
-  (symbol (lib_id "Component_lib:54722-0604") (at 100.33 -93.98 0) (unit 1)
-    (in_bom yes) (on_board yes) (dnp no) (fields_autoplaced)
-    (property "Reference" "J1" (at 110.49 -100.33 0)
-      (effects (font (size 1.27 1.27)))
+  (wire (pts (xy 101.6 68.58) (xy 116.84 68.58))
+    (stroke (width 0) (type default))
+  )
+  (wire (pts (xy 144.78 20.32) (xy 144.78 25.4))
+    (stroke (width 0) (type default))
+  )
+  (wire (pts (xy 114.3 71.12) (xy 101.6 71.12))
+    (stroke (width 0) (type default))
+  )
+  (bus (pts (xy 101.6 73.66) (xy 111.76 73.66))
+    (stroke (width 0) (type default))
+  )
+  (wire (pts (xy 147.32 17.78) (xy 93.98 17.78))
+    (stroke (width 0) (type default))
+  )
+  (wire (pts (xy 147.32 25.4) (xy 147.32 17.78))
+    (stroke (width 0) (type default))
+  )
+  (wire (pts (xy 96.52 20.32) (xy 144.78 20.32))
+    (stroke (width 0) (type default))
+  )
+  (bus (pts (xy 111.76 73.66) (xy 111.76 109.22))
+    (stroke (width 0) (type default))
+  )
+  (wire (pts (xy 91.44 15.24) (xy 149.86 15.24))
+    (stroke (width 0) (type default))
+  )
+  (wire (pts (xy 93.98 17.78) (xy 93.98 25.4))
+    (stroke (width 0) (type default))
+  )
+  (wire (pts (xy 127 106.68) (xy 114.3 106.68))
+    (stroke (width 0) (type default))
+  )
+  (wire (pts (xy 96.52 25.4) (xy 96.52 20.32))
+    (stroke (width 0) (type default))
+  )
+  (bus (pts (xy 111.76 109.22) (xy 127 109.22))
+    (stroke (width 0) (type default))
+  )
+  (wire (pts (xy 91.44 25.4) (xy 91.44 15.24))
+    (stroke (width 0) (type default))
+  )
+  (wire (pts (xy 149.86 15.24) (xy 149.86 25.4))
+    (stroke (width 0) (type default))
+  )
+  (wire (pts (xy 114.3 106.68) (xy 114.3 71.12))
+    (stroke (width 0) (type default))
+  )
+  (wire (pts (xy 116.84 68.58) (xy 116.84 104.14))
+    (stroke (width 0) (type default))
+  )
+  (wire (pts (xy 116.84 104.14) (xy 127 104.14))
+    (stroke (width 0) (type default))
+  )
+  (sheet (at 127 25.4) (size 50.8 50.8) (fields_autoplaced)
+    (stroke (width 0.1524) (type solid))
+    (fill (color 0 0 0 0.0000))
+    (property "Sheetname" "200_1S_Charger" (at 127 24.6884 0)
+      (effects (font (size 1.27 1.27)) (justify left bottom))
     )
-    (property "Value" "54722-0604" (at 110.49 -97.79 0)
-      (effects (font (size 1.27 1.27)))
+    (property "Sheetfile" "1S_Charger.kicad_sch" (at 127 76.7846 0)
+      (effects (font (size 1.27 1.27)) (justify left top))
     )
-    (property "Footprint" "547220604" (at 105.41 -15.24 0)
-      (effects (font (size 1.27 1.27)) (justify left top) hide)
+    (pin "VSYS" output (at 149.86 25.4 90)
+      (effects (font (size 1.27 1.27)) (justify right))
     )
-    (property "Datasheet" "https://componentsearchengine.com/Datasheets/1/54722-0604.pdf" (at 119.38 100.94 0)
-      (effects (font (size 1.27 1.27)) (justify left top) hide)
+    (pin "VBUS" input (at 144.78 25.4 90)
+      (effects (font (size 1.27 1.27)) (justify right))
     )
-    (property "Height" "1.35" (at 119.38 300.94 0)
-      (effects (font (size 1.27 1.27)) (justify left top) hide)
+    (pin "VBAT" bidirectional (at 147.32 25.4 90)
+      (effects (font (size 1.27 1.27)) (justify right))
     )
-    (property "Mouser Part Number" "538-54722-0604" (at 119.38 400.94 0)
-      (effects (font (size 1.27 1.27)) (justify left top) hide)
+    (pin "GND" passive (at 162.56 76.2 270)
+      (effects (font (size 1.27 1.27)) (justify left))
     )
-    (property "Mouser Price/Stock" "https://www.mouser.co.uk/ProductDetail/Molex/54722-0604?qs=OdNwOVlk5%2FhqhipZBZs72A%3D%3D" (at 119.38 500.94 0)
-      (effects (font (size 1.27 1.27)) (justify left top) hide)
-    )
-    (property "Manufacturer_Name" "Molex" (at 119.38 600.94 0)
-      (effects (font (size 1.27 1.27)) (justify left top) hide)
-    )
-    (property "Manufacturer_Part_Number" "54722-0604" (at 119.38 700.94 0)
-      (effects (font (size 1.27 1.27)) (justify left top) hide)
-    )
-    (pin "1")
-    (pin "10")
-    (pin "11")
-    (pin "12")
-    (pin "13")
-    (pin "14")
-    (pin "15")
-    (pin "16")
-    (pin "17")
-    (pin "18")
-    (pin "19")
-    (pin "2")
-    (pin "20")
-    (pin "21")
-    (pin "22")
-    (pin "23")
-    (pin "24")
-    (pin "25")
-    (pin "26")
-    (pin "27")
-    (pin "28")
-    (pin "29")
-    (pin "3")
-    (pin "30")
-    (pin "31")
-    (pin "32")
-    (pin "33")
-    (pin "34")
-    (pin "35")
-    (pin "36")
-    (pin "37")
-    (pin "38")
-    (pin "39")
-    (pin "4")
-    (pin "40")
-    (pin "41")
-    (pin "42")
-    (pin "43")
-    (pin "44")
-    (pin "45")
-    (pin "46")
-    (pin "47")
-    (pin "48")
-    (pin "49")
-    (pin "5")
-    (pin "50")
-    (pin "51")
-    (pin "52")
-    (pin "53")
-    (pin "54")
-    (pin "55")
-    (pin "56")
-    (pin "57")
-    (pin "58")
-    (pin "59")
-    (pin "6")
-    (pin "60")
-    (pin "7")
-    (pin "8")
-    (pin "9")
     (instances
-      (project "ESPSoM_HW00"
-        (path "/14b8af2e-80ef-48c8-890f-5f81b4faa854"
-          (reference "J1") (unit 1)
-        )
+      (project "untitled"
+        (path "/14b8af2e-80ef-48c8-890f-5f81b4faa854" (page "3"))
       )
     )
   )
-  (sheet (at 132.08 67.31) (size 39.37 27.94) (fields_autoplaced)
+  (sheet (at 50.8 25.4) (size 50.8 50.8) (fields_autoplaced)
     (stroke (width 0.1524) (type solid))
     (fill (color 0 0 0 0.0000))
-    (property "Sheetname" "1S_Charger" (at 132.08 66.5984 0)
+    (property "Sheetname" "100_Connectors" (at 50.8 24.6884 0)
       (effects (font (size 1.27 1.27)) (justify left bottom))
     )
-    (property "Sheetfile" "1S_Charger.kicad_sch" (at 132.08 95.8346 0)
+    (property "Sheetfile" "Connectors.kicad_sch" (at 50.8 76.7846 0)
       (effects (font (size 1.27 1.27)) (justify left top))
     )
+    (pin "D-" bidirectional (at 101.6 71.12 0)
+      (effects (font (size 1.27 1.27)) (justify right))
+    )
+    (pin "VBAT" bidirectional (at 93.98 25.4 90)
+      (effects (font (size 1.27 1.27)) (justify right))
+    )
+    (pin "D+" bidirectional (at 101.6 68.58 0)
+      (effects (font (size 1.27 1.27)) (justify right))
+    )
+    (pin "GND" passive (at 86.36 76.2 270)
+      (effects (font (size 1.27 1.27)) (justify left))
+    )
+    (pin "IO[0..42]" bidirectional (at 101.6 73.66 0)
+      (effects (font (size 1.27 1.27)) (justify right))
+    )
+    (pin "VBUS" output (at 96.52 25.4 90)
+      (effects (font (size 1.27 1.27)) (justify right))
+    )
+    (pin "+3V3" input (at 88.9 25.4 90)
+      (effects (font (size 1.27 1.27)) (justify right))
+    )
+    (pin "VSYS" input (at 91.44 25.4 90)
+      (effects (font (size 1.27 1.27)) (justify right))
+    )
     (instances
-      (project "ESPSoM_HW00"
+      (project "untitled"
         (path "/14b8af2e-80ef-48c8-890f-5f81b4faa854" (page "2"))
       )
     )
+  )
+  (sheet (at 127 101.6) (size 50.8 50.8) (fields_autoplaced)
+    (stroke (width 0.1524) (type solid))
+    (fill (color 0 0 0 0.0000))
+    (property "Sheetname" "400_ESP32" (at 127 100.8884 0)
+      (effects (font (size 1.27 1.27)) (justify left bottom))
+    )
+    (property "Sheetfile" "ESP32S2FH4S2.kicad_sch" (at 127 152.9846 0)
+      (effects (font (size 1.27 1.27)) (justify left top))
+    )
+    (pin "D-" bidirectional (at 127 106.68 180)
+      (effects (font (size 1.27 1.27)) (justify left))
+    )
+    (pin "+3V3" input (at 160.02 101.6 90)
+      (effects (font (size 1.27 1.27)) (justify right))
+    )
+    (pin "D+" bidirectional (at 127 104.14 180)
+      (effects (font (size 1.27 1.27)) (justify left))
+    )
+    (pin "GND" passive (at 167.64 152.4 270)
+      (effects (font (size 1.27 1.27)) (justify left))
+    )
+    (pin "IO[0..42]" bidirectional (at 127 109.22 180)
+      (effects (font (size 1.27 1.27)) (justify left))
+    )
+    (instances
+      (project "untitled"
+        (path "/14b8af2e-80ef-48c8-890f-5f81b4faa854" (page "5"))
+      )
+    )
+  )
+  (sheet (at 50.8 101.6) (size 50.8 50.8) (fields_autoplaced)
+    (stroke (width 0.1524) (type solid))
+    (fill (color 0 0 0 0.0000))
+    (property "Sheetname" "300_Power" (at 50.8 100.8884 0)
+      (effects (font (size 1.27 1.27)) (justify left bottom))
+    )
+    (property "Sheetfile" "Power.kicad_sch" (at 50.8 152.9846 0)
+      (effects (font (size 1.27 1.27)) (justify left top))
+    )
+    (pin "+3V3" output (at 88.9 101.6 90)
+      (effects (font (size 1.27 1.27)) (justify right))
+    )
+    (pin "VSYS" input (at 86.36 101.6 90)
+      (effects (font (size 1.27 1.27)) (justify right))
+    )
+    (pin "GND" passive (at 88.9 152.4 270)
+      (effects (font (size 1.27 1.27)) (justify left))
+    )
+    (instances
+      (project "untitled"
+        (path "/14b8af2e-80ef-48c8-890f-5f81b4faa854" (page "4"))
+      )
+    )
