File: Hardware/ESPSoM/ESPSoM_HW00/ESPSoM_HW00/Power.kicad_sch (KiCad schematic)
At the start: 7 parts, among them U301 MIC5528-3.3YMT-T5, U302 MIC5528-3.3YMT-T5

Commit message: schematic first commit
Parts:
- removed C303, C304: 2u2, Capacitor_SMD:C_0603_1608Metric, symbol Component lib:C
- removed U302: MIC5528-3.3YMT-T5, Component_lib:SON40P120X120X60-7N-D, symbol Component lib:MIC5528-3.3YMT-T5
