File: Hardware/ESP_S3_SoM/ESP_S3_SoM_HW00/1S_Charger.kicad_sch (KiCad schematic)
At the start: 14 parts, among them U201 BQ24075RGTR

Commit message: added SPI Bus
Other:
- title: PMK_Keyboard -> PSoM - ESP S3
Changed lines of the file:
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@@
   (paper "A4")
   (title_block
-    (title "PMK_Keyboard")
-    (date "2023-02-06")
+    (title "PSoM - ESP S3")
+    (date "2023-04-17")
     (rev "HW00")
     (company "PumaCorp")
@@
     (pin "1")
     (instances
-      (project "ESPSoM_HW00"
+      (project "ESP_S3_SoM_HW00"
         (path "/14b8af2e-80ef-48c8-890f-5f81b4faa854/a8f40f14-1954-4df1-a27b-4ef4decd9fbc"
           (reference "#PWR0205") (unit 1)
@@
     (pin "")
     (instances
-      (project "ESPSoM_HW00"
+      (project "ESP_S3_SoM_HW00"
         (path "/14b8af2e-80ef-48c8-890f-5f81b4faa854/a8f40f14-1954-4df1-a27b-4ef4decd9fbc"
           (reference "#VBAT0201") (unit 1)
@@
     (pin "1")
     (instances
-      (project "ESPSoM_HW00"
+      (project "ESP_S3_SoM_HW00"
         (path "/14b8af2e-80ef-48c8-890f-5f81b4faa854/a8f40f14-1954-4df1-a27b-4ef4decd9fbc"
           (reference "#PWR0201") (unit 1)
@@
     (pin "2")
     (instances
-      (project "ESPSoM_HW00"
+      (project "ESP_S3_SoM_HW00"
         (path "/14b8af2e-80ef-48c8-890f-5f81b4faa854/a8f40f14-1954-4df1-a27b-4ef4decd9fbc"
           (reference "R202") (unit 1)
@@
     (pin "2")
     (instances
-      (project "ESPSoM_HW00"
+      (project "ESP_S3_SoM_HW00"
         (path "/14b8af2e-80ef-48c8-890f-5f81b4faa854/a8f40f14-1954-4df1-a27b-4ef4decd9fbc"
           (reference "R203") (unit 1)
@@
     (pin "1")
     (instances
-      (project "ESPSoM_HW00"
+      (project "ESP_S3_SoM_HW00"
         (path "/14b8af2e-80ef-48c8-890f-5f81b4faa854/a8f40f14-1954-4df1-a27b-4ef4decd9fbc"
           (reference "TP201") (unit 1)
@@
     (pin "1")
     (instances
-      (project "ESPSoM_HW00"
+      (project "ESP_S3_SoM_HW00"
         (path "/14b8af2e-80ef-48c8-890f-5f81b4faa854/a8f40f14-1954-4df1-a27b-4ef4decd9fbc"
           (reference "#PWR0121") (unit 1)
@@
     (pin "")
     (instances
-      (project "ESPSoM_HW00"
+      (project "ESP_S3_SoM_HW00"
         (path "/14b8af2e-80ef-48c8-890f-5f81b4faa854/a8f40f14-1954-4df1-a27b-4ef4decd9fbc"
           (reference "#VSYS0105") (unit 1)
@@
     (pin "9")
     (instances
-      (project "ESPSoM_HW00"
+      (project "ESP_S3_SoM_HW00"
         (path "/14b8af2e-80ef-48c8-890f-5f81b4faa854/a8f40f14-1954-4df1-a27b-4ef4decd9fbc"
           (reference "U201") (unit 1)
@@
     (pin "2")
     (instances
-      (project "ESPSoM_HW00"
+      (project "ESP_S3_SoM_HW00"
         (path "/14b8af2e-80ef-48c8-890f-5f81b4faa854/a8f40f14-1954-4df1-a27b-4ef4decd9fbc"
           (reference "C203") (unit 1)
@@
     (pin "1")
     (instances
-      (project "ESPSoM_HW00"
+      (project "ESP_S3_SoM_HW00"
         (path "/14b8af2e-80ef-48c8-890f-5f81b4faa854/a8f40f14-1954-4df1-a27b-4ef4decd9fbc"
           (reference "#PWR0209") (unit 1)
@@
     (pin "1")
     (instances
-      (project "ESPSoM_HW00"
+      (project "ESP_S3_SoM_HW00"
         (path "/14b8af2e-80ef-48c8-890f-5f81b4faa854/a8f40f14-1954-4df1-a27b-4ef4decd9fbc"
           (reference "#PWR0208") (unit 1)
@@
     (pin "")
     (instances
-      (project "ESPSoM_HW00"
+      (project "ESP_S3_SoM_HW00"
         (path "/14b8af2e-80ef-48c8-890f-5f81b4faa854/a8f40f14-1954-4df1-a27b-4ef4decd9fbc"
           (reference "#VBAT0103") (unit 1)
@@
     (pin "1")
     (instances
-      (project "ESPSoM_HW00"
+      (project "ESP_S3_SoM_HW00"
         (path "/14b8af2e-80ef-48c8-890f-5f81b4faa854/a8f40f14-1954-4df1-a27b-4ef4decd9fbc"
           (reference "#PWR0206") (unit 1)
@@
     (pin "1")
     (instances
-      (project "ESPSoM_HW00"
+      (project "ESP_S3_SoM_HW00"
         (path "/14b8af2e-80ef-48c8-890f-5f81b4faa854/a8f40f14-1954-4df1-a27b-4ef4decd9fbc"
           (reference "#PWR0124") (unit 1)
@@
     (pin "2")
     (instances
-      (project "ESPSoM_HW00"
+      (project "ESP_S3_SoM_HW00"
         (path "/14b8af2e-80ef-48c8-890f-5f81b4faa854/a8f40f14-1954-4df1-a27b-4ef4decd9fbc"
           (reference "R207") (unit 1)
@@
     (pin "")
     (instances
-      (project "ESPSoM_HW00"
+      (project "ESP_S3_SoM_HW00"
         (path "/14b8af2e-80ef-48c8-890f-5f81b4faa854/a8f40f14-1954-4df1-a27b-4ef4decd9fbc"
           (reference "#VSYS0201") (unit 1)
@@
     (pin "2")
     (instances
-      (project "ESPSoM_HW00"
+      (project "ESP_S3_SoM_HW00"
         (path "/14b8af2e-80ef-48c8-890f-5f81b4faa854/a8f40f14-1954-4df1-a27b-4ef4decd9fbc"
           (reference "C202") (unit 1)
@@
     (pin "1")
     (instances
-      (project "ESPSoM_HW00"
+      (project "ESP_S3_SoM_HW00"
         (path "/14b8af2e-80ef-48c8-890f-5f81b4faa854/a8f40f14-1954-4df1-a27b-4ef4decd9fbc"
           (reference "#PWR0202") (unit 1)
@@
     (pin "2")
     (instances
-      (project "ESPSoM_HW00"
+      (project "ESP_S3_SoM_HW00"
         (path "/14b8af2e-80ef-48c8-890f-5f81b4faa854/a8f40f14-1954-4df1-a27b-4ef4decd9fbc"
           (reference "R201") (unit 1)
@@
     (pin "1")
     (instances
-      (project "ESPSoM_HW00"
+      (project "ESP_S3_SoM_HW00"
         (path "/14b8af2e-80ef-48c8-890f-5f81b4faa854/a8f40f14-1954-4df1-a27b-4ef4decd9fbc"
           (reference "#PWR0123") (unit 1)
@@
     (pin "2")
     (instances
-      (project "ESPSoM_HW00"
+      (project "ESP_S3_SoM_HW00"
         (path "/14b8af2e-80ef-48c8-890f-5f81b4faa854/a8f40f14-1954-4df1-a27b-4ef4decd9fbc"
           (reference "D201") (unit 1)
@@
     (pin "1")
     (instances
-      (project "ESPSoM_HW00"
+      (project "ESP_S3_SoM_HW00"
         (path "/14b8af2e-80ef-48c8-890f-5f81b4faa854/a8f40f14-1954-4df1-a27b-4ef4decd9fbc"
           (reference "#PWR0207") (unit 1)
@@
     (pin "1")
     (instances
-      (project "ESPSoM_HW00"
+      (project "ESP_S3_SoM_HW00"
         (path "/14b8af2e-80ef-48c8-890f-5f81b4faa854/a8f40f14-1954-4df1-a27b-4ef4decd9fbc"
           (reference "#PWR0210") (unit 1)
@@
     (pin "1")
     (instances
-      (project "ESPSoM_HW00"
+      (project "ESP_S3_SoM_HW00"
         (path "/14b8af2e-80ef-48c8-890f-5f81b4faa854/a8f40f14-1954-4df1-a27b-4ef4decd9fbc"
           (reference "#PWR0203") (unit 1)
@@
     (pin "1")
     (instances
-      (project "ESPSoM_HW00"
+      (project "ESP_S3_SoM_HW00"
         (path "/14b8af2e-80ef-48c8-890f-5f81b4faa854/a8f40f14-1954-4df1-a27b-4ef4decd9fbc"
           (reference "#PWR0122") (unit 1)
@@
     (pin "2")
     (instances
-      (project "ESPSoM_HW00"
+      (project "ESP_S3_SoM_HW00"
         (path "/14b8af2e-80ef-48c8-890f-5f81b4faa854/a8f40f14-1954-4df1-a27b-4ef4decd9fbc"
           (reference "R204") (unit 1)
@@
     (pin "")
     (instances
-      (project "ESPSoM_HW00"
+      (project "ESP_S3_SoM_HW00"
         (path "/14b8af2e-80ef-48c8-890f-5f81b4faa854/a8f40f14-1954-4df1-a27b-4ef4decd9fbc"
           (reference "#VSYS0108") (unit 1)
@@
     (pin "2")
     (instances
-      (project "ESPSoM_HW00"
+      (project "ESP_S3_SoM_HW00"
         (path "/14b8af2e-80ef-48c8-890f-5f81b4faa854/a8f40f14-1954-4df1-a27b-4ef4decd9fbc"
           (reference "R206") (unit 1)
@@
     (pin "2")
     (instances
-      (project "ESPSoM_HW00"
+      (project "ESP_S3_SoM_HW00"
         (path "/14b8af2e-80ef-48c8-890f-5f81b4faa854/a8f40f14-1954-4df1-a27b-4ef4decd9fbc"
           (reference "C201") (unit 1)
@@
     (pin "2")
     (instances
-      (project "ESPSoM_HW00"
+      (project "ESP_S3_SoM_HW00"
         (path "/14b8af2e-80ef-48c8-890f-5f81b4faa854/a8f40f14-1954-4df1-a27b-4ef4decd9fbc"
           (reference "R205") (unit 1)
@@
     (pin "")
     (instances
-      (project "ESPSoM_HW00"
+      (project "ESP_S3_SoM_HW00"
         (path "/14b8af2e-80ef-48c8-890f-5f81b4faa854/a8f40f14-1954-4df1-a27b-4ef4decd9fbc"
           (reference "#VBAT0202") (unit 1)
@@
     (pin "")
     (instances
-      (project "ESPSoM_HW00"
+      (project "ESP_S3_SoM_HW00"
         (path "/14b8af2e-80ef-48c8-890f-5f81b4faa854/a8f40f14-1954-4df1-a27b-4ef4decd9fbc"
           (reference "#VSYS0107") (unit 1)
@@
     (pin "")
     (instances
-      (project "ESPSoM_HW00"
+      (project "ESP_S3_SoM_HW00"
         (path "/14b8af2e-80ef-48c8-890f-5f81b4faa854/a8f40f14-1954-4df1-a27b-4ef4decd9fbc"
           (reference "#VSYS0106") (unit 1)
@@
     (pin "2")
     (instances
-      (project "ESPSoM_HW00"
+      (project "ESP_S3_SoM_HW00"
         (path "/14b8af2e-80ef-48c8-890f-5f81b4faa854/a8f40f14-1954-4df1-a27b-4ef4decd9fbc"
           (reference "D202") (unit 1)
@@
     (pin "1")
     (instances
-      (project "ESPSoM_HW00"
+      (project "ESP_S3_SoM_HW00"
         (path "/14b8af2e-80ef-48c8-890f-5f81b4faa854/a8f40f14-1954-4df1-a27b-4ef4decd9fbc"
           (reference "#PWR0204") (unit 1)
