File: Hardware/ESP_S3_SoM/ESP_S3_SoM_HW00/Connectors.kicad_sch (KiCad schematic)
At the start: 4 parts, among them J1 54722-0604, J101 USB4510-03-1-A

Commit message: added SPI Bus
Parts:
- J1: footprint 547220604 -> Component_lib:547220604
Connections:
- net RX0: now reaches J1.13
- net TX0: now reaches J1.15
Other:
- title: PMK_Keyboard -> PSoM - ESP S3
