File: Hardware/ESP_S3_SoM/ESP_S3_SoM_HW00/Power.kicad_sch (KiCad schematic)
At the start: 4 parts, among them U301 MIC5528-3.3YMT-T5

Commit message: added SPI Bus
Other:
- title: PMK_Keyboard -> PSoM - ESP S3
Changed lines of the file:
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@@
   (paper "A4")
   (title_block
-    (title "PMK_Keyboard")
-    (date "2023-02-06")
+    (title "PSoM - ESP S3")
+    (date "2023-04-17")
     (rev "HW00")
     (company "PumaCorp")
@@
     (pin "1")
     (instances
-      (project "ESPSoM_HW00"
+      (project "ESP_S3_SoM_HW00"
         (path "/14b8af2e-80ef-48c8-890f-5f81b4faa854/fe763027-4af8-431c-8c5f-e79d70169837"
           (reference "#PWR0303") (unit 1)
@@
     (pin "1")
     (instances
-      (project "ESPSoM_HW00"
+      (project "ESP_S3_SoM_HW00"
         (path "/14b8af2e-80ef-48c8-890f-5f81b4faa854/fe763027-4af8-431c-8c5f-e79d70169837"
           (reference "#PWR0305") (unit 1)
@@
     (pin "1")
     (instances
-      (project "ESPSoM_HW00"
+      (project "ESP_S3_SoM_HW00"
         (path "/14b8af2e-80ef-48c8-890f-5f81b4faa854/fe763027-4af8-431c-8c5f-e79d70169837"
           (reference "#PWR0301") (unit 1)
@@
     (pin "")
     (instances
-      (project "ESPSoM_HW00"
+      (project "ESP_S3_SoM_HW00"
         (path "/14b8af2e-80ef-48c8-890f-5f81b4faa854/fe763027-4af8-431c-8c5f-e79d70169837"
           (reference "#VSYS0103") (unit 1)
@@
     (pin "1")
     (instances
-      (project "ESPSoM_HW00"
+      (project "ESP_S3_SoM_HW00"
         (path "/14b8af2e-80ef-48c8-890f-5f81b4faa854/fe763027-4af8-431c-8c5f-e79d70169837"
           (reference "#PWR0307") (unit 1)
@@
     (pin "1")
     (instances
-      (project "ESPSoM_HW00"
+      (project "ESP_S3_SoM_HW00"
         (path "/14b8af2e-80ef-48c8-890f-5f81b4faa854/fe763027-4af8-431c-8c5f-e79d70169837"
           (reference "#PWR0308") (unit 1)
@@
     (pin "")
     (instances
-      (project "ESPSoM_HW00"
+      (project "ESP_S3_SoM_HW00"
         (path "/14b8af2e-80ef-48c8-890f-5f81b4faa854/fe763027-4af8-431c-8c5f-e79d70169837"
           (reference "#VSYS0104") (unit 1)
@@
     (pin "7")
     (instances
-      (project "ESPSoM_HW00"
+      (project "ESP_S3_SoM_HW00"
         (path "/14b8af2e-80ef-48c8-890f-5f81b4faa854/fe763027-4af8-431c-8c5f-e79d70169837"
           (reference "U301") (unit 1)
@@
     (pin "")
     (instances
-      (project "ESPSoM_HW00"
+      (project "ESP_S3_SoM_HW00"
         (path "/14b8af2e-80ef-48c8-890f-5f81b4faa854/fe763027-4af8-431c-8c5f-e79d70169837"
           (reference "#VSYS0102") (unit 1)
@@
     (pin "2")
     (instances
-      (project "ESPSoM_HW00"
+      (project "ESP_S3_SoM_HW00"
         (path "/14b8af2e-80ef-48c8-890f-5f81b4faa854/fe763027-4af8-431c-8c5f-e79d70169837"
           (reference "C302") (unit 1)
@@
     (pin "2")
     (instances
-      (project "ESPSoM_HW00"
+      (project "ESP_S3_SoM_HW00"
         (path "/14b8af2e-80ef-48c8-890f-5f81b4faa854/fe763027-4af8-431c-8c5f-e79d70169837"
           (reference "R301") (unit 1)
@@
     (pin "2")
     (instances
-      (project "ESPSoM_HW00"
+      (project "ESP_S3_SoM_HW00"
         (path "/14b8af2e-80ef-48c8-890f-5f81b4faa854/fe763027-4af8-431c-8c5f-e79d70169837"
           (reference "C301") (unit 1)
@@
     (pin "1")
     (instances
-      (project "ESPSoM_HW00"
+      (project "ESP_S3_SoM_HW00"
         (path "/14b8af2e-80ef-48c8-890f-5f81b4faa854/fe763027-4af8-431c-8c5f-e79d70169837"
           (reference "#PWR0306") (unit 1)
@@
     (pin "1")
     (instances
-      (project "ESPSoM_HW00"
+      (project "ESP_S3_SoM_HW00"
         (path "/14b8af2e-80ef-48c8-890f-5f81b4faa854/fe763027-4af8-431c-8c5f-e79d70169837"
           (reference "#PWR0304") (unit 1)
@@
     (pin "1")
     (instances
-      (project "ESPSoM_HW00"
+      (project "ESP_S3_SoM_HW00"
         (path "/14b8af2e-80ef-48c8-890f-5f81b4faa854/fe763027-4af8-431c-8c5f-e79d70169837"
           (reference "#PWR0309") (unit 1)
