File: Hardware/ESP_S2_SoM/ESP_S2_SoM_HW00/ESP32S2FH4S2.kicad_sch (KiCad schematic)
At the start: 31 parts, among them SW401 SW_Push, SW402 SW_Push, U401 ESP32-S2FH4, Y601 Crystal_GND24_Small

Commit message: lots of work on routing
Parts:
- C403, C404, C405, C408, C411, C412, C414, C415, C416: footprint Capacitor_SMD:C_0402_1005Metric -> Capacitor_SMD:C_0201_0603Metric
Connections:
- net at C401.1, R401.1: now also Y601.3; no longer Y601.1
- net at C402.1, U401.52 (XTAL_N): now also Y601.1; no longer Y601.3
- net SPICLK renamed SPI2
- net SPICS0 renamed SPI3
- net SPICS1 renamed SPI7
- net SPID renamed SPI0
- net SPIHD renamed SPI5
- net SPIQ renamed SPI1
- net SPIWP renamed SPI4
- net VDD_SPI renamed SPI6
Changed lines of the file:
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@@
+    (stroke (width 0) (type default))
+  )
+  (wire (pts (xy 205.74 45.72) (xy 213.36 45.72))
     (stroke (width 0) (type default))
   )
@@
     (stroke (width 0) (type default))
   )
-  (wire (pts (xy 210.82 45.72) (xy 213.36 45.72))
-    (stroke (width 0) (type default))
-  )
   (wire (pts (xy 241.3 40.64) (xy 243.84 40.64))
     (stroke (width 0) (type default))
@@
     (stroke (width 0) (type default))
   )
-  (wire (pts (xy 210.82 38.1) (xy 213.36 38.1))
+  (wire (pts (xy 205.74 38.1) (xy 213.36 38.1))
     (stroke (width 0) (type default))
   )
@@
     (stroke (width 0) (type default))
   )
-  (wire (pts (xy 210.82 30.48) (xy 213.36 30.48))
+  (wire (pts (xy 205.74 30.48) (xy 213.36 30.48))
     (stroke (width 0) (type default))
   )
@@
     (stroke (width 0) (type default))
   )
+  (wire (pts (xy 205.74 43.18) (xy 213.36 43.18))
+    (stroke (width 0) (type default))
+  )
   (wire (pts (xy 73.66 165.1) (xy 93.98 165.1))
     (stroke (width 0) (type default))
   )
-  (wire (pts (xy 210.82 35.56) (xy 213.36 35.56))
+  (wire (pts (xy 205.74 35.56) (xy 213.36 35.56))
     (stroke (width 0) (type default))
   )
@@
     (stroke (width 0) (type default))
   )
-  (wire (pts (xy 210.82 40.64) (xy 213.36 40.64))
+  (wire (pts (xy 205.74 40.64) (xy 213.36 40.64))
     (stroke (width 0) (type default))
   )
@@
     (stroke (width 0) (type default))
   )
-  (wire (pts (xy 210.82 48.26) (xy 213.36 48.26))
+  (wire (pts (xy 205.74 48.26) (xy 213.36 48.26))
     (stroke (width 0) (type default))
   )
@@
     (stroke (width 0) (type default))
   )
-  (wire (pts (xy 210.82 33.02) (xy 213.36 33.02))
+  (wire (pts (xy 205.74 33.02) (xy 213.36 33.02))
     (stroke (width 0) (type default))
   )
@@
   )
   (wire (pts (xy 241.3 63.5) (xy 243.84 63.5))
-    (stroke (width 0) (type default))
-  )
-  (wire (pts (xy 210.82 43.18) (xy 213.36 43.18))
     (stroke (width 0) (type default))
   )
@@
     (effects (font (size 1.27 1.27)) (justify right bottom))
   )
+  (label "SPI0" (at 213.36 30.48 180) (fields_autoplaced)
+    (effects (font (size 1.27 1.27)) (justify right bottom))
+  )
   (label "IO12" (at 86.36 154.94 270) (fields_autoplaced)
     (effects (font (size 1.27 1.27)) (justify right bottom))
@@
     (effects (font (size 1.27 1.27)) (justify right bottom))
   )
-  (label "SPICLK" (at 210.82 35.56 180) (fields_autoplaced)
+  (label "SPICLK" (at 205.74 35.56 180) (fields_autoplaced)
+    (effects (font (size 1.27 1.27)) (justify right bottom))
+  )
+  (label "SPI1" (at 213.36 33.02 180) (fields_autoplaced)
     (effects (font (size 1.27 1.27)) (justify right bottom))
   )
@@
     (effects (font (size 1.27 1.27)) (justify right bottom))
   )
+  (label "SPI5" (at 213.36 43.18 180) (fields_autoplaced)
+    (effects (font (size 1.27 1.27)) (justify right bottom))
+  )
   (label "IO10" (at 81.28 154.94 270) (fields_autoplaced)
     (effects (font (size 1.27 1.27)) (justify right bottom))
@@
     (effects (font (size 1.27 1.27)) (justify left bottom))
   )
-  (label "SPIHD" (at 210.82 43.18 180) (fields_autoplaced)
+  (label "SPIHD" (at 205.74 43.18 180) (fields_autoplaced)
     (effects (font (size 1.27 1.27)) (justify right bottom))
   )
@@
     (effects (font (size 1.27 1.27)) (justify left bottom))
   )
-  (label "SPICS1" (at 210.82 48.26 180) (fields_autoplaced)
+  (label "SPICS1" (at 205.74 48.26 180) (fields_autoplaced)
     (effects (font (size 1.27 1.27)) (justify right bottom))
   )
@@
     (effects (font (size 1.27 1.27)) (justify right bottom))
   )
-  (label "SPIQ" (at 210.82 33.02 180) (fields_autoplaced)
+  (label "SPIQ" (at 205.74 33.02 180) (fields_autoplaced)
     (effects (font (size 1.27 1.27)) (justify right bottom))
   )
@@
     (effects (font (size 1.27 1.27)) (justify right bottom))
   )
-  (label "SPICS0" (at 210.82 38.1 180) (fields_autoplaced)
+  (label "SPI4" (at 213.36 40.64 180) (fields_autoplaced)
+    (effects (font (size 1.27 1.27)) (justify right bottom))
+  )
+  (label "SPICS0" (at 205.74 38.1 180) (fields_autoplaced)
     (effects (font (size 1.27 1.27)) (justify right bottom))
   )
@@
     (effects (font (size 1.27 1.27)) (justify left bottom))
   )
+  (label "SPI3" (at 213.36 38.1 180) (fields_autoplaced)
+    (effects (font (size 1.27 1.27)) (justify right bottom))
+  )
   (label "IO21" (at 114.3 154.94 270) (fields_autoplaced)
     (effects (font (size 1.27 1.27)) (justify right bottom))
@@
     (effects (font (size 1.27 1.27)) (justify right bottom))
   )
+  (label "SPI2" (at 213.36 35.56 180) (fields_autoplaced)
+    (effects (font (size 1.27 1.27)) (justify right bottom))
+  )
   (label "IO15" (at 96.52 154.94 270) (fields_autoplaced)
     (effects (font (size 1.27 1.27)) (justify right bottom))
   )
+  (label "SPI7" (at 213.36 48.26 180) (fields_autoplaced)
+    (effects (font (size 1.27 1.27)) (justify right bottom))
+  )
   (label "IO1" (at 66.04 119.38 180) (fields_autoplaced)
     (effects (font (size 1.27 1.27)) (justify right bottom))
@@
     (effects (font (size 1.27 1.27)) (justify left bottom))
   )
-  (label "SPIWP" (at 210.82 40.64 180) (fields_autoplaced)
+  (label "SPIWP" (at 205.74 40.64 180) (fields_autoplaced)
     (effects (font (size 1.27 1.27)) (justify right bottom))
   )
@@
     (effects (font (size 1.27 1.27)) (justify right bottom))
   )
-  (label "VDD_SPI" (at 210.82 45.72 180) (fields_autoplaced)
+  (label "VDD_SPI" (at 205.74 45.72 180) (fields_autoplaced)
     (effects (font (size 1.27 1.27)) (justify right bottom))
   )
@@
     (effects (font (size 1.27 1.27)) (justify right bottom))
   )
+  (label "SPI6" (at 213.36 45.72 180) (fields_autoplaced)
+    (effects (font (size 1.27 1.27)) (justify right bottom))
+  )
   (label "IO34" (at 241.3 76.2 180) (fields_autoplaced)
     (effects (font (size 1.27 1.27)) (justify right bottom))
@@
     (effects (font (size 1.27 1.27)) (justify left bottom))
   )
-  (label "SPID" (at 210.82 30.48 180) (fields_autoplaced)
+  (label "SPID" (at 205.74 30.48 180) (fields_autoplaced)
     (effects (font (size 1.27 1.27)) (justify right bottom))
   )
@@
       (effects (font (size 1.27 1.27)) (justify left))
     )
-    (property "Footprint" "Capacitor_SMD:C_0402_1005Metric" (at 127.9652 175.26 0)
+    (property "Footprint" "Capacitor_SMD:C_0201_0603Metric" (at 127.9652 175.26 0)
       (effects (font (size 1.27 1.27)) hide)
     )
@@
       (effects (font (size 1.27 1.27)) (justify left))
     )
-    (property "Footprint" "Capacitor_SMD:C_0402_1005Metric" (at 54.3052 101.6 0)
+    (property "Footprint" "Capacitor_SMD:C_0201_0603Metric" (at 54.3052 101.6 0)
       (effects (font (size 1.27 1.27)) hide)
     )
@@
       (effects (font (size 1.27 1.27)) (justify left))
     )
-    (property "Footprint" "Capacitor_SMD:C_0402_1005Metric" (at 171.1452 144.78 0)
+    (property "Footprint" "Capacitor_SMD:C_0201_0603Metric" (at 171.1452 144.78 0)
       (effects (font (size 1.27 1.27)) hide)
     )
@@
       (effects (font (size 1.27 1.27)) (justify left))
     )
-    (property "Footprint" "Capacitor_SMD:C_0402_1005Metric" (at 145.7452 147.32 0)
+    (property "Footprint" "Capacitor_SMD:C_0201_0603Metric" (at 145.7452 147.32 0)
       (effects (font (size 1.27 1.27)) hide)
     )
@@
       (effects (font (size 1.27 1.27)) (justify left))
     )
-    (property "Footprint" "Capacitor_SMD:C_0402_1005Metric" (at 33.9852 93.98 0)
+    (property "Footprint" "Capacitor_SMD:C_0201_0603Metric" (at 33.9852 93.98 0)
       (effects (font (size 1.27 1.27)) hide)
     )
@@
       (effects (font (size 1.27 1.27)) (justify left))
     )
-    (property "Footprint" "Capacitor_SMD:C_0402_1005Metric" (at 74.6252 175.26 0)
+    (property "Footprint" "Capacitor_SMD:C_0201_0603Metric" (at 74.6252 175.26 0)
       (effects (font (size 1.27 1.27)) hide)
     )
@@
       (effects (font (size 1.27 1.27)) (justify left))
     )
-    (property "Footprint" "Capacitor_SMD:C_0402_1005Metric" (at 145.7452 91.44 0)
+    (property "Footprint" "Capacitor_SMD:C_0201_0603Metric" (at 145.7452 91.44 0)
       (effects (font (size 1.27 1.27)) hide)
     )
@@
     )
   )
-  (symbol (lib_id "Device:Crystal_GND24_Small") (at 91.44 63.5 0) (unit 1)
-    (in_bom yes) (on_board yes) (dnp no) (fields_autoplaced)
-    (property "Reference" "Y601" (at 103.7063 60.8457 0)
-      (effects (font (size 1.27 1.27)))
-    )
-    (property "Value" "Crystal_GND24_Small" (at 103.7063 62.7667 0)
+  (symbol (lib_id "Device:Crystal_GND24_Small") (at 91.44 63.5 0) (mirror y) (unit 1)
+    (in_bom yes) (on_board yes) (dnp no)
+    (property "Reference" "Y601" (at 79.1737 60.8457 0)
+      (effects (font (size 1.27 1.27)))
+    )
+    (property "Value" "Crystal_GND24_Small" (at 79.1737 62.7667 0)
       (effects (font (size 1.27 1.27)))
     )
@@
       (effects (font (size 1.27 1.27)) (justify left))
     )
-    (property "Footprint" "Capacitor_SMD:C_0402_1005Metric" (at 44.1452 93.98 0)
+    (property "Footprint" "Capacitor_SMD:C_0201_0603Metric" (at 44.1452 93.98 0)
       (effects (font (size 1.27 1.27)) hide)
     )
@@
       (effects (font (size 1.27 1.27)) (justify left))
     )
-    (property "Footprint" "Capacitor_SMD:C_0402_1005Metric" (at 54.3052 121.92 0)
-      (effects (font (size 1.27 1.27)) hide)
-    )
+    (property "Footprint" "Capacitor_SMD:C_0201_0603Metric" (at 54.3052 121.92 0)
+      (effects (font (size 1.27 1.27)) hide)
+    )

Commit message: led footprint update
Parts:
- D401: footprint Component_lib:LED_0402_1005Metric_DUALSIDE -> LED_SMD:LED_0402_1005Metric
Changed lines of the file:
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@@
       (effects (font (size 1.27 1.27)) (justify right))
     )
-    (property "Footprint" "Component_lib:LED_0402_1005Metric_DUALSIDE" (at 205.74 90.17 0)
+    (property "Footprint" "LED_SMD:LED_0402_1005Metric" (at 205.74 90.17 0)
       (effects (font (size 1.27 1.27)) hide)
     )
