File: Hardware/ESP_S2_SoM/ESP_S2_SoM_HW00/_autosave-ESP_S2_SoM_HW00.kicad_pcb (KiCad board)
At the start: 6 copper layers, 29.5 x 24.7 mm, 55 parts, among them J1 DF40C-60DP-0.4V(51), J2 Bare PCB USB C, SW401 SW_Push, SW402 SW_Push, U201 BQ24075RGTR, U301 MIC5528-3.3YMT-T5, U401 ESP32-S2FH4, Y601 Crystal_GND24_Small

Commit message: Little backup before messing up everything
Parts:
- moved C401 2.96 mm to (127.5, 91.8), turned to 180 degrees
- moved Y601 2.25 mm to (127.5, 93.4), turned to 90 degrees
- moved C402 2.07 mm to (127.5, 95.0), turned to 0 degrees
- moved C405 0.33 mm to (130.2, 93.9), turned to 180 degrees
Routing:
- net Net-(U401-XTAL_N): track 5.15 -> 0.67 mm
- net Net-(U401-XTAL_P): track 1.13 -> 0.00 mm
- net +3V3: track 11.5 -> 10.5 mm
- net Net-(C401-Pad1): track 1.98 -> 1.00 mm
- net GND: vias 31 -> 11
