File: Hardware/ESP_S2_SoM/ESP_S2_SoM_HW00/_autosave-Connectors.kicad_sch (KiCad schematic)
At the start: 4 parts, among them J1 DF40C-60DP-0.4V(51), J2 Bare PCB USB C

Commit message: Little backup before messing up everything
Connections:
- net IO42: now also J1.52; no longer J1.48
- net RX0: now also J1.50; no longer J1.52
- net TX0: now also J1.48; no longer J1.50
Changed lines of the file:
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@@
     (effects (font (size 1.27 1.27)) (justify left bottom))
   )
-  (label "IO42" (at 175.26 114.3 0) (fields_autoplaced)
+  (label "IO42" (at 175.26 119.38 0) (fields_autoplaced)
     (effects (font (size 1.27 1.27)) (justify left bottom))
   )
@@
     (effects (font (size 1.27 1.27)) (justify left bottom))
   )
-  (label "RX0" (at 175.26 119.38 0) (fields_autoplaced)
+  (label "RX0" (at 175.26 116.84 0) (fields_autoplaced)
     (effects (font (size 1.27 1.27)) (justify left bottom))
   )
-  (label "TX0" (at 175.26 116.84 0) (fields_autoplaced)
+  (label "TX0" (at 175.26 114.3 0) (fields_autoplaced)
     (effects (font (size 1.27 1.27)) (justify left bottom))
   )
