File: Hardware/ESP_S2_SoM/ESP_S2_SoM_HW00/Power.kicad_sch (KiCad schematic)
At the start: 4 parts, among them U301 MIC5528-3.3YMT-T5

Commit message: Small cartouche mistake
Other:
- title: PSoM - ESP S3 -> PSoM - ESP S2
Changed lines of the file:
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@@
   (paper "A4")
   (title_block
-    (title "PSoM - ESP S3")
+    (title "PSoM - ESP S2")
     (date "2023-04-17")
     (rev "HW00")
