File: Hardware/PSoM_RP2040/PSoM_RP2040_00/1S_Charger.kicad_sch (KiCad schematic)
At the start: 15 parts, among them U301 BQ24075RGTR

Commit message: updated bas de page
Other:
- title: PSoM - ESP S3 -> PSoM - RP2040
Changed lines of the file:
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@@
   (paper "A4")
   (title_block
-    (title "PSoM - ESP S3")
-    (date "2023-04-17")
+    (title "PSoM - RP2040")
+    (date "2024-02-28")
     (rev "HW00")
     (company "PumaCorp")
