File: Hardware/PSoM_RP2040/PSoM_RP2040_00/Power.kicad_sch (KiCad schematic)
At the start: 4 parts, among them U401 MIC5528-3.3YMT-T5

Commit message: updated bas de page
Other:
- title: PSoM - ESP S3 -> PSoM - RP2040
Changed lines of the file:
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@@
   (paper "A4")
   (title_block
-    (title "PSoM - ESP S3")
-    (date "2023-04-17")
+    (title "PSoM - RP2040")
+    (date "2024-02-28")
     (rev "HW00")
     (company "PumaCorp")
