File: Hardware/PSoM_RP2040/PSoM_RP2040_00/RP2040.kicad_sch (KiCad schematic)
At the start: 26 parts, among them SW501 SW_Push, SW502 SW_Push, U501 SC0914_7_, U502 W25Q128JVPIQ_TR, Y501 830105420809

Commit message: updated bas de page
Other:
- title: PSoM - ESP32 S2 -> PSoM - RP2040
Changed lines of the file:
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@@
   (paper "A4")
   (title_block
-    (title "PSoM - ESP32 S2")
-    (date "2023-04-17")
+    (title "PSoM - RP2040")
+    (date "2024-02-28")
     (rev "HW00")
     (company "PumaCorp")
