File: Hardware/PSoM_RP2040/PSoM_RP2040_00/PSoM_RP2040_00.kicad_sch (KiCad schematic)
At the start: 0 parts

Commit message: updated bas de page
Other:
- title: PSoM - ESP S3 -> PSoM - RP2040
Changed lines of the file:
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@@
   (paper "A4")
   (title_block
-    (title "PSoM - ESP S3")
-    (date "2023-04-17")
+    (title "PSoM - RP2040")
+    (date "2024-02-28")
     (rev "HW00")
     (company "PumaCorp")

Commit message: small adjustements on rp2040 routing
Other:
- sheet 200_Connectors renamed 100_Connectors
Changed lines of the file:
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@@
     (stroke (width 0.1524) (type solid))
     (fill (color 0 0 0 0.0000))
-    (property "Sheetname" "200_Connectors" (at 50.8 24.6884 0)
+    (property "Sheetname" "100_Connectors" (at 50.8 24.6884 0)
       (effects (font (size 1.27 1.27)) (justify left bottom))
     )
