File: Hardware/ESP32_PicoD4_SOM/ESP32_PicoD4_SoM_HW00/ESP32S2FH4S2.kicad_sch (KiCad schematic)
At the start: 21 parts, among them SW401 SW_Push, SW402 SW_Push, U401 ESP32-PICO-D4

Commit message: First version of schematic Connections
Done according to definition in pinout.xlsx (available on master)
Renaming ESP_... to ESP32_...
Parts:
- renumbered C406 to C403, C407 to C404, R402 to R401, R401 to R402, R405 to R403, R407 to R404, R409 to R405, R403 to R406, R406 to R407, R410 to R409, R404 to R410, SW402 to SW401, SW401 to SW402
Connections:
- net IO15: no longer R401.1
- net IO16: no longer U401.27 (GPIO17), U401.34 (GPIO5)
- net IO17: now also U401.27 (GPIO17)
- net IO23: now also R401.1
- net IO36: now also U401.5 (SENSOR_VP/GPIO36)
- net IO37: now also U401.6 (SENSOR_CAPP/GPIO37)
- net IO38: now also U401.7 (SENSOR_CAPN/GPIO38)
- net IO39: now also U401.8 (SENSOR_VN/GPIO39)
- net IO5: now also U401.34 (GPIO5)
- net LNA_IN renamed LAN_IN
Other:
- note added: "(alone)U0TXD debug"
- note added: "(together)SDIO Slave Timing"
- note added: "VDD_SDIO Ctrl"
- moved on the sheet: C405, R402, R403, R404, R405, R406, R407, R408, R409, R410, SW401, SW402
