File: Hardware/ESP32_PicoD4_SOM/ESP32_PicoD4_SoM_HW00/ESP_PicoD4_SoM_HW00.kicad_sch (KiCad schematic)
At the start: 0 parts

Commit message: First version of schematic Connections
Done according to definition in pinout.xlsx (available on master)
Renaming ESP_... to ESP32_...
Other:
- sheet 100_Connectors ports: added IO[0..39], SPI[0..6]; removed D+, D-, IO[0..42], SPI[0..7]
- sheet 400_ESP32 ports: added IO[0..39], SPI[0..6]; removed D+, D-, IO[0..42], SPI[0..7]
Changed lines of the file:
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@@
-    (stroke (width 0) (type default))
-  )
-  (wire (pts (xy 121.92 58.42) (xy 101.6 58.42))
     (stroke (width 0) (type default))
   )
@@
     (stroke (width 0) (type default))
   )
-  (wire (pts (xy 121.92 58.42) (xy 121.92 104.14))
-    (stroke (width 0) (type default))
-  )
   (wire (pts (xy 111.76 114.3) (xy 111.76 68.58))
     (stroke (width 0) (type default))
@@
     (stroke (width 0) (type default))
   )
-  (wire (pts (xy 119.38 106.68) (xy 127 106.68))
-    (stroke (width 0) (type default))
-  )
   (bus (pts (xy 114.3 66.04) (xy 114.3 111.76))
     (stroke (width 0) (type default))
@@
     (stroke (width 0) (type default))
   )
-  (wire (pts (xy 119.38 60.96) (xy 119.38 106.68))
-    (stroke (width 0) (type default))
-  )
   (bus (pts (xy 101.6 66.04) (xy 114.3 66.04))
     (stroke (width 0) (type default))
   )
-  (wire (pts (xy 101.6 60.96) (xy 119.38 60.96))
-    (stroke (width 0) (type default))
-  )
   (bus (pts (xy 116.84 63.5) (xy 101.6 63.5))
     (stroke (width 0) (type default))
@@
   )
   (wire (pts (xy 88.9 22.86) (xy 88.9 25.4))
-    (stroke (width 0) (type default))
-  )
-  (wire (pts (xy 127 104.14) (xy 121.92 104.14))
     (stroke (width 0) (type default))
   )
@@
       (effects (font (size 1.27 1.27)) (justify left top))
     )
-    (pin "D-" bidirectional (at 101.6 60.96 0)
-      (effects (font (size 1.27 1.27)) (justify right))
-    )
     (pin "VBAT" bidirectional (at 93.98 25.4 90)
       (effects (font (size 1.27 1.27)) (justify right))
     )
-    (pin "D+" bidirectional (at 101.6 58.42 0)
-      (effects (font (size 1.27 1.27)) (justify right))
-    )
     (pin "GND" passive (at 91.44 76.2 270)
       (effects (font (size 1.27 1.27)) (justify left))
     )
-    (pin "IO[0..42]" bidirectional (at 101.6 63.5 0)
+    (pin "IO[0..39]" bidirectional (at 101.6 63.5 0)
       (effects (font (size 1.27 1.27)) (justify right))
     )
@@
       (effects (font (size 1.27 1.27)) (justify right))
     )
-    (pin "SPI[0..7]" bidirectional (at 101.6 66.04 0)
+    (pin "SPI[0..6]" bidirectional (at 101.6 66.04 0)
       (effects (font (size 1.27 1.27)) (justify right))
     )
@@
       (effects (font (size 1.27 1.27)) (justify left top))
     )
-    (pin "D-" bidirectional (at 127 106.68 180)
-      (effects (font (size 1.27 1.27)) (justify left))
-    )
     (pin "+3V3" input (at 160.02 101.6 90)
       (effects (font (size 1.27 1.27)) (justify right))
     )
-    (pin "D+" bidirectional (at 127 104.14 180)
-      (effects (font (size 1.27 1.27)) (justify left))
-    )
     (pin "GND" passive (at 167.64 152.4 270)
       (effects (font (size 1.27 1.27)) (justify left))
     )
-    (pin "IO[0..42]" bidirectional (at 127 109.22 180)
+    (pin "IO[0..39]" bidirectional (at 127 109.22 180)
       (effects (font (size 1.27 1.27)) (justify left))
     )
@@
       (effects (font (size 1.27 1.27)) (justify left))
     )
-    (pin "SPI[0..7]" bidirectional (at 127 111.76 180)
-      (effects (font (size 1.27 1.27)) (justify left))
-    )
+    (pin "SPI[0..6]" bidirectional (at 127 111.76 180)
+      (effects (font (size 1.27 1.27)) (justify left))
+    )
