File: Hardware/PSoM_nRF52840/PSoM_nRF52840_HW00/PSoM_nRF52840_HW00/Connectors.kicad_sch (KiCad schematic)
At the start: 7 parts, among them J101 DF40C-60DP-0.4V(51), J102 Bare PCB USB C

Commit message: nrf schematic ongoing
Parts:
- renumbered C415 to C101
Changed lines of the file:
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@@
 		(dnp no)
 		(fields_autoplaced yes)
-		(property "Reference" "C415"
+		(property "Reference" "C101"
 			(at 231.521 130.1663 0)
 			(effects
@@
 					(unit 1)
 				)
-				(path "/14b8af2e-80ef-48c8-890f-5f81b4faa854/f80064c8-41de-40ac-b331-44fdb69dca18"
-					(reference "C415")
-					(unit 1)
-				)

Commit message: working on schematic
Other:
- title: PSoM - ESP S3 -> PSoM - nRF52840
Changed lines of the file:
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@@
 	(paper "A4")
 	(title_block
-		(title "PSoM - ESP S3")
-		(date "2023-04-17")
+		(title "PSoM - nRF52840")
+		(date "2024-09-30")
 		(rev "HW00")
 		(company "PumaCorp")
