File: Hardware/PSoM_nRF52840/PSoM_nRF52840_HW00/PSoM_nRF52840_HW00/1S_Charger.kicad_sch (KiCad schematic)
At the start: 15 parts, among them U201 BQ24075RGTR

Commit message: working on schematic
Parts:
- removed C201, C203: 4u7, Capacitor_SMD:C_0603_1608Metric, symbol Component lib:C
- removed C202: 1u, Capacitor_SMD:C_0603_1608Metric, symbol Component lib:C
- removed R1, R2: R, Resistor_SMD:R_0402_1005Metric, symbol Component_lib:R
- removed R201: 0, Resistor_SMD:R_0402_1005Metric, symbol Component_lib:R
- removed R202: 36k5, Resistor_SMD:R_0402_1005Metric, symbol Component_lib:R
- removed R203: 590, Resistor_SMD:R_0402_1005Metric, symbol Component_lib:R
- removed R204: 1k1, Resistor_SMD:R_0402_1005Metric, symbol Component_lib:R
- removed R207: 100k, Resistor_SMD:R_0402_1005Metric, symbol Component_lib:R
- removed U201: BQ24075RGTR, Component_lib:QFN50P300X300X100-17N-D, symbol Component lib:BQ24075RGTR
- added U2: NPM1300-QEAA-R, Component_lib:NPM1300-QEAA-R, symbol Component_lib:NPM1300-QEAA-R
Other:
- note removed: "1550/Iin=R502"
- note removed: "1u to 10u"
- note removed: "36k5: 5h safety 30min pre charge"
- note removed: "4u7 to 47u"
- note removed: "890/Ichg=R503"
- note removed: "SYSOFF low for normal operation"
- title: PSoM - ESP S3 -> PSoM - nRF52840

Commit message: power organisation thinking
Parts:
- added C2, C3: C, symbol Component_lib:C
- added L3, L4: L, symbol Component_lib:L
- added R1: 250k, symbol Component_lib:R
- added R2: 0, symbol Component_lib:R
- added SHIPHLD: TestPoint, symbol Connector:TestPoint
Connections:
- net GND: now also U2.33 (PAD), R1.2, R2.2
- net SDA: now reaches U2.13 (SDA)
- net SCL: now reaches U2.14 (SCL)
- net at U2.15 (SHPHLD): now also SHIPHLD.1
- net at U2.16 (VSET2): now also R1.1
- net at U2.17 (VSET1): now also R2.1
