File: Hardware/PSoM_nRF52840/PSoM_nRF52840_00/nRF52840.kicad_sch (KiCad schematic)
At the start: 33 parts, among them U1 nRF52840-QIAA-aQFN73, Y1 830108161301

Commit message: working on nrf52840
Parts:
- removed SW?: SW_Push, Component_lib:B3U-1000P, symbol Switch:SW_Push
- C413: now not fitted
- L?: value L -> 4n7
- renumbered C1 to C451, L1 to L451, L2 to L452, U1 to U401, Y1 to Y401
Connections:
- net EN is gone; now on net SPI3: C?.1, R?.2, SW?.1
- net DCC: now also U401.B3 (DCC)
- net SPI0: now also U401.AD22 (TRACEDATA0/P1.00)
- net SPI1: now also U401.AD18 (P0.22)
- net SPI2: now also U401.AC15 (P0.19)
- net SPI3: now also U401.AC13 (P0.18/~{RESET})
- net SPI4: now also U401.AC19 (P0.23)
- net SPI5: now also U401.AC17 (P0.21)
- net SPI7: now also U401.AD16 (P0.20)
- net P25: now reaches U401.A10 (AIN5/P0.29)
- net VBAT_VOLTAGE_DIVIDER: now reaches U401.A12 (AIN0/P0.02)
- net P33: now reaches U401.A14 (P1.15)
- net P29: now reaches U401.A16 (P1.13)
- net P23: now reaches U401.A20 (P1.10)
- net P27: now reaches U401.A8 (AIN7/P0.31)
- net P38: now reaches U401.AC11 (P0.16)
- net P44: now reaches U401.AC21 (P0.25)
- net P34: now reaches U401.AC9 (P0.14)
- net P36: now reaches U401.AD10 (P0.15)
- net P40: now reaches U401.AD12 (P0.17)
- net P42: now reaches U401.AD20 (P0.24)
- net P17: now reaches U401.B9 (AIN6/P0.30)
- net P13: now reaches U401.D2 (XL1/P0.00)
- net P15: now reaches U401.F2 (XL2/P0.01)
- net P30: now reaches U401.G1 (P0.26)
- net P32: now reaches U401.H2 (P0.27)
- net P19: now reaches U401.J1 (AIN2/P0.04)
- net P21: now reaches U401.K2 (AIN3/P0.05)
- net P5: now reaches U401.L1 (P0.06)
- net P7: now reaches U401.M2 (TRACECLK/P0.07)
- net P9: now reaches U401.N1 (P0.08)
- net P11: now reaches U401.P2 (P1.08)
- net P39: now reaches U401.R1 (TRACEDATA3/P1.09)
- net P35: now reaches U401.T2 (TRACEDATA2/P0.11)
- net P37: now reaches U401.U1 (TRACEDATA1/P0.12)
- net P31: now reaches U401.U24 (P1.04)
- net P52: now reaches U401.W24 (P1.02)
- net P46: now reaches U401.Y23 (P1.01)
- net IO15: no longer names the net of R?.1
- net SDWDIO renamed SWDIO
- no-connect marks 0 -> 1
Other:
- note added: "50mA"
- note added: "A22"
- note added: "AD14"
- note added: "AD23"
- note added: "ADC"
- note added: "B1"
- note added: "B5"
- note added: "I2C"
- note added: "LF"
- note added: "QSPI"
- note added: "W1/Y2"
- note removed: "Boot mode"
- note removed: "Strapping pins"
- moved on the sheet: ANT?, C405, C406, C407, C408, C409, C410, C411, C412, C414, C415, C416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

Commit message: footprint assignement done
Parts:
- C401, C402, C405, C407, C408, C409, C411, C412: footprint (none) -> Capacitor_SMD:C_0201_0603Metric
- C406, C420, C421: footprint (none) -> Capacitor_SMD:C_0603_1608Metric
- C410, C413, C414, C415, C416: footprint (none) -> Capacitor_SMD:C_0402_1005Metric
- L402: footprint (none) -> Inductor_SMD:L_0603_1608Metric
- L403: footprint (none) -> Inductor_SMD:L_0402_1005Metric
Connections:
- no-connect marks 1 -> 11
Changed lines of the file:
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@@
 	)
 	(no_connect
+		(at 50.8 137.16)
+	)
+	(no_connect
+		(at 50.8 129.54)
+	)
+	(no_connect
+		(at 50.8 119.38)
+	)
+	(no_connect
+		(at 50.8 109.22)
+	)
+	(no_connect
+		(at 111.76 99.06)
+	)
+	(no_connect
 		(at 93.98 60.96)
 	)
+	(no_connect
+		(at 50.8 116.84)
+	)
+	(no_connect
+		(at 50.8 132.08)
+	)
+	(no_connect
+		(at 111.76 73.66)
+	)
+	(no_connect
+		(at 50.8 114.3)
+	)
+	(no_connect
+		(at 111.76 134.62)
+	)
 	(bus_entry
 		(at 251.46 86.36)
@@
 	(wire
 		(pts
+			(xy 269.24 15.24) (xy 271.78 15.24)
+		)
+		(stroke
+			(width 0)
+			(type default)
+		)
+	)
+	(wire
+		(pts
 			(xy 248.92 40.64) (xy 251.46 40.64)
 		)
@@
 	(wire
 		(pts
-			(xy 111.76 73.66) (xy 114.3 73.66)
-		)
-		(stroke
-			(width 0)
-			(type default)
-		)
-	)
-	(wire
-		(pts
 			(xy 269.24 53.34) (xy 271.78 53.34)
 		)
@@
 		)
 	)
+	(label "VBAT_VOLTAGE_DIVIDER"
+		(at 269.24 15.24 180)
+		(fields_autoplaced yes)
+		(effects
+			(font
+				(size 1.27 1.27)
+			)
+			(justify right bottom)
+		)
+	)
 	(label "P31"
 		(at 48.26 111.76 180)
@@
 		)
 	)
+	(hierarchical_label "VBAT_VOLTAGE_DIVIDER"
+		(shape input)
+		(at 271.78 15.24 0)
+		(fields_autoplaced yes)
+		(effects
+			(font
+				(size 1.27 1.27)
+			)
+			(justify left)
+		)
+	)
 	(hierarchical_label "VDD_nRF"
 		(shape input)
@@
 			)
 		)
-		(property "Footprint" ""
+		(property "Footprint" "Capacitor_SMD:C_0603_1608Metric"
 			(at 155.9052 144.78 0)
 			(effects
@@
 			)
 		)
-		(property "Footprint" ""
+		(property "Footprint" "Capacitor_SMD:C_0402_1005Metric"
 			(at 150.8252 172.72 0)
 			(effects
@@
 			)
 		)
-		(property "Footprint" ""
+		(property "Footprint" "Capacitor_SMD:C_0402_1005Metric"
 			(at 125.4252 172.72 0)
 			(effects
@@
 			)
 		)
-		(property "Footprint" ""
+		(property "Footprint" "Capacitor_SMD:C_0201_0603Metric"
 			(at 206.7052 119.38 0)
 			(effects
@@
 			)
 		)
-		(property "Footprint" ""
+		(property "Footprint" "Capacitor_SMD:C_0603_1608Metric"
 			(at 155.9052 119.38 0)
 			(effects
@@
 			)
 		)
-		(property "Footprint" ""
+		(property "Footprint" "Capacitor_SMD:C_0402_1005Metric"
 			(at 206.7052 144.78 0)
 			(effects
@@
 			)
 		)
-		(property "Footprint" ""
+		(property "Footprint" "Capacitor_SMD:C_0201_0603Metric"
 			(at 163.5252 172.72 0)
 			(effects
@@
 			)
 		)
-		(property "Footprint" ""
+		(property "Footprint" "Capacitor_SMD:C_0201_0603Metric"
 			(at 89.8652 185.42 0)
 			(effects
@@
 			)
 		)
-		(property "Footprint" ""
+		(property "Footprint" "Capacitor_SMD:C_0201_0603Metric"
 			(at 181.3052 119.38 0)
 			(effects
@@
 			)
 		)
-		(property "Footprint" ""
+		(property "Footprint" "Capacitor_SMD:C_0603_1608Metric"
 			(at 168.6052 119.38 0)
 			(effects
@@
 			)
 		)
-		(property "Footprint" ""
+		(property "Footprint" "Capacitor_SMD:C_0402_1005Metric"
 			(at 194.0052 119.38 0)
 			(effects
@@
 			)
 		)
-		(property "Footprint" ""
+		(property "Footprint" "Capacitor_SMD:C_0201_0603Metric"
 			(at 105.1052 185.42 0)
 			(effects
@@
 			)
 		)
-		(property "Footprint" ""
+		(property "Footprint" "Capacitor_SMD:C_0201_0603Metric"
 			(at 168.6052 144.78 0)
 			(effects
@@
 			)
 		)
-		(property "Footprint" ""
+		(property "Footprint" "Capacitor_SMD:C_0201_0603Metric"
 			(at 181.3052 144.78 0)
 			(effects
@@
 			)
 		)
-		(property "Footprint" ""
+		(property "Footprint" "Capacitor_SMD:C_0402_1005Metric"
 			(at 138.1252 172.72 0)
 			(effects
@@
 			)
 		)
-		(property "Footprint" ""
+		(property "Footprint" "Capacitor_SMD:C_0201_0603Metric"
 			(at 194.0052 144.78 0)
 			(effects
@@
 			)
 		)
-		(property "Footprint" ""
+		(property "Footprint" "Inductor_SMD:L_0402_1005Metric"
 			(at 156.21 190.5 90)
 			(effects
@@
 			)
 		)
-		(property "Footprint" ""
+		(property "Footprint" "Inductor_SMD:L_0603_1608Metric"
 			(at 146.05 190.5 90)
 			(effects

Commit message: working on schematic
Connections:
- net SPI3 renamed RESET
- net VBAT_VOLTAGE_DIVIDER: no longer names the net of U401.A12 (AIN0/P0.02)

Commit message: added nfc connector + update pinout info
Parts:
- added J401, J402: Conn_01x01_Pin, Connector_Wire:SolderWirePad_1x01_SMD_1x2mm, symbol Connector:Conn_01x01_Pin
Connections:
- net NFC2: now reaches U401.J24 (NFC2/P0.10)
- net NFC2: now also J402.1 (Pin_1)
- net NFC1: now reaches U401.L24 (NFC1/P0.09)
- net NFC1: now also J401.1 (Pin_1)
- no-connect marks 11 -> 12
Changed lines of the file:
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@@
 	)
 	(no_connect
+		(at 111.76 71.12)
+	)
+	(no_connect
 		(at 50.8 129.54)
 	)
@@
 	(wire
 		(pts
+			(xy 53.34 172.72) (xy 50.8 172.72)
+		)
+		(stroke
+			(width 0)
+			(type default)
+		)
+	)
+	(wire
+		(pts
 			(xy 48.26 101.6) (xy 50.8 101.6)
 		)
@@
 	(wire
 		(pts
+			(xy 111.76 91.44) (xy 114.3 91.44)
+		)
+		(stroke
+			(width 0)
+			(type default)
+		)
+	)
+	(wire
+		(pts
 			(xy 111.76 139.7) (xy 114.3 139.7)
 		)
@@
 	(wire
 		(pts
-			(xy 111.76 71.12) (xy 114.3 71.12)
-		)
-		(stroke
-			(width 0)
-			(type default)
-		)
-	)
-	(wire
-		(pts
 			(xy 137.16 160.02) (xy 137.16 162.56)
 		)
@@
 	(wire
 		(pts
+			(xy 111.76 88.9) (xy 114.3 88.9)
+		)
+		(stroke
+			(width 0)
+			(type default)
+		)
+	)
+	(wire
+		(pts
 			(xy 269.24 48.26) (xy 271.78 48.26)
 		)
@@
 		)
 	)
+	(wire
+		(pts
+			(xy 53.34 170.18) (xy 50.8 170.18)
+		)
+		(stroke
+			(width 0)
+			(type default)
+		)
+	)
 	(bus
 		(pts
@@
 		)
 	)
-	(label "NFC"
+	(label "NFC2"
 		(at 114.3 91.44 0)
 		(fields_autoplaced yes)
@@
 		)
 	)
+	(label "NFC1"
+		(at 53.34 170.18 0)
+		(fields_autoplaced yes)
+		(effects
+			(font
+				(size 1.27 1.27)
+			)
+			(justify left bottom)
+		)
+	)
 	(label "P7"
 		(at 248.92 25.4 180)
@@
 		)
 	)
-	(label "NFC"
+	(label "NFC1"
 		(at 114.3 88.9 0)
 		(fields_autoplaced yes)
@@
 		)
 	)
+	(label "NFC2"
+		(at 53.34 172.72 0)
+		(fields_autoplaced yes)
+		(effects
+			(font
+				(size 1.27 1.27)
+			)
+			(justify left bottom)
+		)
+	)
 	(label "P42"
 		(at 248.92 83.82 180)
@@
 	)
 	(symbol
+		(lib_id "Connector:Conn_01x01_Pin")
+		(at 45.72 172.72 0)
+		(mirror x)
+		(unit 1)
+		(exclude_from_sim no)
+		(in_bom yes)
+		(on_board yes)
+		(dnp no)
+		(property "Reference" "J402"
+			(at 46.355 177.0322 0)
+			(effects
+				(font
+					(size 1.27 1.27)
+				)
+			)
+		)
+		(property "Value" "Conn_01x01_Pin"
+			(at 46.355 174.5469 0)
+			(effects
+				(font
+					(size 1.27 1.27)
+				)
+			)
+		)
+		(property "Footprint" "Connector_Wire:SolderWirePad_1x01_SMD_1x2mm"
+			(at 45.72 172.72 0)
+			(effects
+				(font
+					(size 1.27 1.27)
+				)
+				(hide yes)
+			)
+		)
+		(property "Datasheet" "~"
+			(at 45.72 172.72 0)
+			(effects
+				(font
+					(size 1.27 1.27)
+				)
+				(hide yes)
+			)
+		)
+		(property "Description" "Generic connector, single row, 01x01, script generated"
+			(at 45.72 172.72 0)
+			(effects
+				(font
+					(size 1.27 1.27)
+				)
+				(hide yes)
+			)
+		)
+		(pin "1"
+		)
+		(instances
+			(project "PSoM_nRF52840_00"
+				(path "/14b8af2e-80ef-48c8-890f-5f81b4faa854/f0612286-54f9-458a-949b-e71e3a4da5eb"
+					(reference "J402")
+					(unit 1)
+				)
+			)
+		)
+	)
+	(symbol
 		(lib_id "Component lib:C")
 		(at 167.64 83.82 0)
@@
 					(unit 1)
 				)
+			)
+		)
+	)
+	(symbol
+		(lib_id "Connector:Conn_01x01_Pin")
+		(at 45.72 170.18 0)
+		(unit 1)
+		(exclude_from_sim no)
+		(in_bom yes)
+		(on_board yes)
+		(dnp no)
+		(fields_autoplaced yes)
+		(property "Reference" "J401"
+			(at 46.355 165.8678 0)
+			(effects
+				(font
+					(size 1.27 1.27)
+				)
+			)
+		)
+		(property "Value" "Conn_01x01_Pin"
+			(at 46.355 168.3531 0)
+			(effects
+				(font
+					(size 1.27 1.27)
+				)
+			)
+		)
+		(property "Footprint" "Connector_Wire:SolderWirePad_1x01_SMD_1x2mm"
+			(at 45.72 170.18 0)
+			(effects
+				(font
+					(size 1.27 1.27)
+				)
+				(hide yes)
+			)
+		)
+		(property "Datasheet" "~"
+			(at 45.72 170.18 0)
+			(effects
+				(font
+					(size 1.27 1.27)
+				)
+				(hide yes)
+			)
+		)
+		(property "Description" "Generic connector, single row, 01x01, script generated"
+			(at 45.72 170.18 0)
+			(effects
+				(font
+					(size 1.27 1.27)
+				)
+				(hide yes)
+			)
+		)
+		(pin "1"
+		)
+		(instances
+			(project ""
+				(path "/14b8af2e-80ef-48c8-890f-5f81b4faa854/f0612286-54f9-458a-949b-e71e3a4da5eb"
+					(reference "J401")
+					(unit 1)
+				)

Commit message: routing is doing great progress
Changed lines of the file:
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@@
 	(wire
 		(pts
-			(xy 223.52 38.1) (xy 231.14 38.1)
-		)
-		(stroke
-			(width 0)
-			(type default)
-		)
-	)
-	(wire
-		(pts
 			(xy 248.92 48.26) (xy 251.46 48.26)
 		)
@@
 	(wire
 		(pts
+			(xy 213.36 38.1) (xy 231.14 38.1)
+		)
+		(stroke
+			(width 0)
+			(type default)
+		)
+	)
+	(wire
+		(pts
 			(xy 180.34 134.62) (xy 193.04 134.62)
 		)
@@
 		)
 	)
+	(label "VDD_nRF"
+		(at 213.36 38.1 180)
+		(effects
+			(font
+				(size 1.27 1.27)
+			)
+			(justify right bottom)
+		)
+	)
 	(label "DCC"
 		(at 139.7 190.5 180)
@@
 		(on_board yes)
 		(dnp no)
-		(fields_autoplaced yes)
 		(property "Reference" "C421"
 			(at 171.45 114.2999 0)

Commit message: schematic should be done
Parts:
- removed ANT?: 2450AT18A100E, Component_lib:ANTC3216X140N, symbol Component lib:2450AT18A100E
- added ANT450: 2450AT18A100E, Component_lib:ANTC3216X140N, symbol Component_lib:2450AT18A100E
Connections:
- net ANT_OUT: now also ANT450.1
- net DCC_DEC4: now reaches L402.2, L403.1
- net P13 renamed SDA
- net P15 renamed SCL
Other:
- moved on the sheet: L403

Commit message: working on the routing
Connections:
- net +3V3 is gone; now on net VDD_nRF: R?.1
- net P35: now also U401.U1 (TRACEDATA1/P0.12); no longer U401.T2 (TRACEDATA2/P0.11)
- net P37: now also U401.T2 (TRACEDATA2/P0.11); no longer U401.U1 (TRACEDATA1/P0.12)
Changed lines of the file:
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@@
+		)
+	)
+	(label "P36"
+		(at 121.92 106.68 0)
+		(fields_autoplaced yes)
+		(effects
+			(font
+				(size 1.27 1.27)
+			)
+			(justify left bottom)
 		)
 	)
@@
 		)
 	)
+	(label "P38"
+		(at 121.92 104.14 0)
+		(fields_autoplaced yes)
+		(effects
+			(font
+				(size 1.27 1.27)
+			)
+			(justify left bottom)
+		)
+	)
 	(label "P17"
 		(at 248.92 38.1 180)
@@
 		)
 	)
+	(label "VDD_nRF"
+		(at 241.3 124.46 180)
+		(fields_autoplaced yes)
+		(effects
+			(font
+				(size 1.27 1.27)
+			)
+			(justify right bottom)
+		)
+	)
 	(label "P40"
 		(at 248.92 81.28 180)
@@
 	)
 	(label "P37"
-		(at 114.3 96.52 0)
+		(at 114.3 93.98 0)
 		(fields_autoplaced yes)
 		(effects
@@
 	)
 	(label "P35"
-		(at 114.3 93.98 0)
+		(at 114.3 96.52 0)
 		(fields_autoplaced yes)
 		(effects
@@
 					(unit 1)
 				)
-			)
-		)
-	)
-	(symbol
-		(lib_id "power:+3V3")
-		(at 241.3 124.46 0)
-		(unit 1)
-		(exclude_from_sim no)
-		(in_bom yes)
-		(on_board yes)
-		(dnp no)
-		(fields_autoplaced yes)
-		(property "Reference" "#PWR?"
-			(at 241.3 128.27 0)
-			(effects
-				(font
-					(size 1.27 1.27)
-				)
-				(hide yes)
-			)
-		)
-		(property "Value" "+3V3"
-			(at 241.3 120.8842 0)
-			(effects
-				(font
-					(size 1.27 1.27)
-				)
-			)
-		)
-		(property "Footprint" ""
-			(at 241.3 124.46 0)
-			(effects
-				(font
-					(size 1.27 1.27)
-				)
-				(hide yes)
-			)
-		)
-		(property "Datasheet" ""
-			(at 241.3 124.46 0)
-			(effects
-				(font
-					(size 1.27 1.27)
-				)
-				(hide yes)
-			)
-		)
-		(property "Description" ""
-			(at 241.3 124.46 0)
-			(effects
-				(font
-					(size 1.27 1.27)
-				)
-				(hide yes)
-			)
-		)
-		(pin "1"
-		)
-		(instances
-			(project "nRF52840"
-				(path "/1055a12c-de3d-4753-aef1-2b6e803dd877"
-					(reference "#PWR?")
-					(unit 1)
-				)
-			)
-			(project "nRF52840"
-				(path "/14b8af2e-80ef-48c8-890f-5f81b4faa854/f0612286-54f9-458a-949b-e71e3a4da5eb"
-					(reference "#PWR0109")
-					(unit 1)
-				)
-			)
-			(project "PMK_Keyboard"
-				(path "/c3b08055-08a5-4979-9bf8-f36ab0917722/38b3fafb-a86a-4dac-a282-53c1331aa596"
-					(reference "#PWR0421")
-					(unit 1)
-				)
