File: Hardware/PSoM_nRF52840/PSoM_nRF52840_00/1S_Charger.kicad_sch (KiCad schematic)
At the start: 17 parts, among them U201 NPM1300-QEAA-R

Commit message: moved the nrf away and re routed everything
Connections:
- net SCL renamed P15
- net SDA renamed P13
Changed lines of the file:
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@@
 		(at 124.46 96.52)
 	)
+	(bus_entry
+		(at 266.7 76.2)
+		(size 2.54 -2.54)
+		(stroke
+			(width 0)
+			(type default)
+		)
+	)
+	(bus_entry
+		(at 266.7 73.66)
+		(size 2.54 -2.54)
+		(stroke
+			(width 0)
+			(type default)
+		)
+	)
 	(wire
 		(pts
@@
 	(wire
 		(pts
-			(xy 266.7 73.66) (xy 269.24 73.66)
-		)
-		(stroke
-			(width 0)
-			(type default)
-		)
-	)
-	(wire
-		(pts
 			(xy 236.22 68.58) (xy 233.68 68.58)
 		)
@@
 	(wire
 		(pts
-			(xy 269.24 78.74) (xy 266.7 78.74)
+			(xy 269.24 81.28) (xy 266.7 81.28)
 		)
 		(stroke
@@
 	(wire
 		(pts
-			(xy 266.7 78.74) (xy 266.7 81.28)
+			(xy 266.7 81.28) (xy 266.7 83.82)
 		)
 		(stroke
@@
 		)
 	)
+	(bus
+		(pts
+			(xy 269.24 68.58) (xy 269.24 71.12)
+		)
+		(stroke
+			(width 0)
+			(type default)
+		)
+	)
 	(wire
 		(pts
@@
 		)
 	)
+	(bus
+		(pts
+			(xy 269.24 71.12) (xy 269.24 73.66)
+		)
+		(stroke
+			(width 0)
+			(type default)
+		)
+	)
 	(wire
 		(pts
@@
 	(wire
 		(pts
+			(xy 264.16 73.66) (xy 266.7 73.66)
+		)
+		(stroke
+			(width 0)
+			(type default)
+		)
+	)
+	(wire
+		(pts
 			(xy 162.56 106.68) (xy 167.64 106.68)
 		)
@@
 	(wire
 		(pts
-			(xy 266.7 68.58) (xy 269.24 68.58)
-		)
-		(stroke
-			(width 0)
-			(type default)
-		)
-	)
-	(wire
-		(pts
 			(xy 162.56 99.06) (xy 167.64 99.06)
 		)
@@
 		(pts
 			(xy 162.56 71.12) (xy 165.1 71.12)
+		)
+		(stroke
+			(width 0)
+			(type default)
+		)
+	)
+	(wire
+		(pts
+			(xy 264.16 76.2) (xy 266.7 76.2)
 		)
 		(stroke
@@
 		)
 	)
-	(label "SDA"
-		(at 266.7 73.66 180)
-		(effects
-			(font
-				(size 1.27 1.27)
-			)
-			(justify right bottom)
-		)
-	)
 	(label "VSET1"
 		(at 106.68 111.76 0)
@@
 		)
 	)
+	(label "P13"
+		(at 121.92 127 180)
+		(effects
+			(font
+				(size 1.27 1.27)
+			)
+			(justify right bottom)
+		)
+	)
+	(label "P15"
+		(at 121.92 124.46 180)
+		(effects
+			(font
+				(size 1.27 1.27)
+			)
+			(justify right bottom)
+		)
+	)
 	(label "VBUS_OUT"
 		(at 266.7 33.02 180)
@@
 		)
 	)
+	(label "P13"
+		(at 264.16 73.66 180)
+		(effects
+			(font
+				(size 1.27 1.27)
+			)
+			(justify right bottom)
+		)
+	)
 	(label "LED0"
 		(at 121.92 101.6 180)
@@
 		)
 	)
-	(label "SCL"
-		(at 266.7 68.58 180)
-		(effects
-			(font
-				(size 1.27 1.27)
-			)
-			(justify right bottom)
-		)
-	)
 	(label "3V3_nRF"
 		(at 266.7 48.26 180)
@@
 		)
 	)
-	(label "SDA"
-		(at 121.92 127 180)
+	(label "P15"
+		(at 264.16 76.2 180)
 		(effects
 			(font
@@
 			)
 			(justify left bottom)
-		)
-	)
-	(label "SCL"
-		(at 121.92 124.46 180)
-		(effects
-			(font
-				(size 1.27 1.27)
-			)
-			(justify right bottom)
 		)
 	)
@@
 		)
 	)
-	(hierarchical_label "SCL"
-		(shape input)
-		(at 269.24 68.58 0)
-		(effects
-			(font
-				(size 1.27 1.27)
-			)
-			(justify left)
-		)
-	)
 	(hierarchical_label "VBAT"
 		(shape bidirectional)
@@
 		)
 	)
+	(hierarchical_label "P[0..52]"
+		(shape bidirectional)
+		(at 269.24 68.58 0)
+		(effects
+			(font
+				(size 1.27 1.27)
+			)
+			(justify left)
+		)
+	)
 	(hierarchical_label "GND"
 		(shape passive)
-		(at 269.24 78.74 0)
-		(effects
-			(font
-				(size 1.27 1.27)
-			)
-			(justify left)
-		)
-	)
-	(hierarchical_label "SDA"
-		(shape bidirectional)
-		(at 269.24 73.66 0)
+		(at 269.24 81.28 0)
 		(effects
 			(font
@@
 	(symbol
 		(lib_id "power:GND")
-		(at 266.7 81.28 0)
+		(at 266.7 83.82 0)
 		(unit 1)
 		(exclude_from_sim no)
@@
 		(fields_autoplaced yes)
 		(property "Reference" "#PWR0202"
-			(at 266.7 87.63 0)
+			(at 266.7 90.17 0)
 			(effects
 				(font
@@
 		)
 		(property "Value" "GND"
-			(at 266.7 85.7234 0)
+			(at 266.7 88.2634 0)
 			(effects
 				(font
@@
 		)
 		(property "Footprint" ""
-			(at 266.7 81.28 0)
+			(at 266.7 83.82 0)
 			(effects
 				(font
@@
 		)
 		(property "Datasheet" ""
-			(at 266.7 81.28 0)
+			(at 266.7 83.82 0)
 			(effects
 				(font
@@
 		)
 		(property "Description" ""
-			(at 266.7 81.28 0)
-			(effects
-				(font
+			(at 266.7 83.82 0)
+			(effects
+				(font

Commit message: TODO: RF and GND vias
Parts:
- removed SHIPHLD1: TestPoint, TestPoint:TestPoint_Pad_D1.0mm, symbol Connector:TestPoint
- added R205: 10k, Resistor_SMD:R_0201_0603Metric, symbol Component_lib:R
Connections:
- net GND: now also R205.2
- net SHIP: now also R205.1
Other:
- moved on the sheet: R203, R204
Changed lines of the file:
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@@
+	(wire
+		(pts
+			(xy 106.68 121.92) (xy 106.68 119.38)
+		)
+		(stroke
+			(width 0)
+			(type default)
+		)
+	)
 	(wire
 		(pts
@@
 	(wire
 		(pts
-			(xy 91.44 111.76) (xy 124.46 111.76)
+			(xy 83.82 111.76) (xy 124.46 111.76)
 		)
 		(stroke
@@
 	(wire
 		(pts
-			(xy 91.44 116.84) (xy 91.44 111.76)
+			(xy 83.82 116.84) (xy 83.82 111.76)
 		)
 		(stroke
@@
 	(wire
 		(pts
-			(xy 111.76 119.38) (xy 124.46 119.38)
-		)
-		(stroke
-			(width 0)
-			(type default)
-		)
-	)
-	(wire
-		(pts
-			(xy 101.6 124.46) (xy 101.6 127)
+			(xy 106.68 119.38) (xy 124.46 119.38)
+		)
+		(stroke
+			(width 0)
+			(type default)
+		)
+	)
+	(wire
+		(pts
+			(xy 93.98 124.46) (xy 93.98 127)
 		)
 		(stroke
@@
 	(wire
 		(pts
-			(xy 91.44 124.46) (xy 91.44 127)
+			(xy 83.82 124.46) (xy 83.82 127)
 		)
 		(stroke
@@
 	(wire
 		(pts
-			(xy 101.6 114.3) (xy 101.6 116.84)
+			(xy 93.98 114.3) (xy 93.98 116.84)
 		)
 		(stroke
@@
 	(wire
 		(pts
+			(xy 106.68 129.54) (xy 106.68 132.08)
+		)
+		(stroke
+			(width 0)
+			(type default)
+		)
+	)
+	(wire
+		(pts
 			(xy 165.1 116.84) (xy 165.1 121.92)
 		)
@@
 	(wire
 		(pts
-			(xy 124.46 114.3) (xy 101.6 114.3)
+			(xy 124.46 114.3) (xy 93.98 114.3)
 		)
 		(stroke
@@
 	(text_box "Only REG2 is capable of outputing 3V3 with resistor setup\n47k = 1V8 on VREG1\n250k-500k = 3V3 on VREG2\n"
 		(exclude_from_sim no)
-		(at 71.12 137.16 0)
+		(at 71.12 139.7 0)
 		(size 60.96 7.62)
 		(stroke
@@
 	(text "Has to be between\n250k and 500k,\nInventory has 470k"
 		(exclude_from_sim no)
-		(at 104.14 124.46 0)
+		(at 96.52 124.46 0)
 		(effects
 			(font
@@
 		(lib_name "GND_1")
 		(lib_id "power:GND")
-		(at 101.6 127 0)
+		(at 93.98 127 0)
 		(unit 1)
 		(exclude_from_sim no)
@@
 		(fields_autoplaced yes)
 		(property "Reference" "#PWR024"
-			(at 101.6 133.35 0)
+			(at 93.98 133.35 0)
 			(effects
 				(font
@@
 		)
 		(property "Value" "GND"
-			(at 101.6 132.08 0)
+			(at 93.98 132.08 0)
 			(effects
 				(font
@@
 		)
 		(property "Footprint" ""
-			(at 101.6 127 0)
+			(at 93.98 127 0)
 			(effects
 				(font
@@
 		)
 		(property "Datasheet" ""
-			(at 101.6 127 0)
+			(at 93.98 127 0)
 			(effects
 				(font
@@
 		)
 		(property "Description" "Power symbol creates a global label with name \"GND\" , ground"
-			(at 101.6 127 0)
+			(at 93.98 127 0)
 			(effects
 				(font
@@
 	)
 	(symbol
+		(lib_id "Component_lib:R")
+		(at 106.68 121.92 0)
+		(unit 1)
+		(exclude_from_sim no)
+		(in_bom yes)
+		(on_board yes)
+		(dnp no)
+		(property "Reference" "R205"
+			(at 109.22 124.4599 0)
+			(effects
+				(font
+					(size 1.27 1.27)
+				)
+				(justify left)
+			)
+		)
+		(property "Value" "10k"
+			(at 109.22 126.9999 0)
+			(effects
+				(font
+					(size 1.27 1.27)
+				)
+				(justify left)
+			)
+		)
+		(property "Footprint" "Resistor_SMD:R_0201_0603Metric"
+			(at 104.902 125.73 90)
+			(effects
+				(font
+					(size 1.27 1.27)
+				)
+				(hide yes)
+			)
+		)
+		(property "Datasheet" "~"
+			(at 106.68 125.73 0)
+			(effects
+				(font
+					(size 1.27 1.27)
+				)
+				(hide yes)
+			)
+		)
+		(property "Description" "Resistor"
+			(at 106.68 121.92 0)
+			(effects
+				(font
+					(size 1.27 1.27)
+				)
+				(hide yes)
+			)
+		)
+		(pin "2"
+		)
+		(pin "1"
+		)
+		(instances
+			(project "PSoM_nRF52840_00"
+				(path "/14b8af2e-80ef-48c8-890f-5f81b4faa854/a8f40f14-1954-4df1-a27b-4ef4decd9fbc"
+					(reference "R205")
+					(unit 1)
+				)
+			)
+		)
+	)
+	(symbol
 		(lib_name "GND_1")
 		(lib_id "power:GND")
@@
 	)
 	(symbol
-		(lib_id "Connector:TestPoint")
-		(at 111.76 119.38 0)
+		(lib_name "GND_1")
+		(lib_id "power:GND")
+		(at 106.68 132.08 0)
 		(unit 1)
 		(exclude_from_sim no)
@@
 		(on_board yes)
 		(dnp no)
-		(property "Reference" "SHIPHLD1"
-			(at 114.3 116.84 0)
-			(effects
-				(font
-					(size 1.27 1.27)
-				)
-				(justify left)
-			)
-		)
-		(property "Value" "TestPoint"
-			(at 114.3 116.84 0)
-			(effects
-				(font
-					(size 1.27 1.27)
-				)
-				(justify left)
-				(hide yes)
-			)
-		)
-		(property "Footprint" "TestPoint:TestPoint_Pad_D1.0mm"
-			(at 116.84 119.38 0)
-			(effects
-				(font
-					(size 1.27 1.27)
-				)
-				(hide yes)
-			)
-		)
-		(property "Datasheet" "~"
-			(at 116.84 119.38 0)
-			(effects
-				(font
-					(size 1.27 1.27)
-				)
-				(hide yes)
-			)
-		)
-		(property "Description" "test point"
-			(at 111.76 119.38 0)
+		(fields_autoplaced yes)
+		(property "Reference" "#PWR011"
+			(at 106.68 138.43 0)
+			(effects
+				(font
+					(size 1.27 1.27)
+				)
+				(hide yes)
+			)
+		)
+		(property "Value" "GND"
+			(at 106.68 137.16 0)
+			(effects
+				(font
+					(size 1.27 1.27)
+				)
+			)
+		)
+		(property "Footprint" ""
+			(at 106.68 132.08 0)
+			(effects
+				(font
+					(size 1.27 1.27)
+				)
+				(hide yes)
+			)
+		)
+		(property "Datasheet" ""
+			(at 106.68 132.08 0)
+			(effects
+				(font
+					(size 1.27 1.27)
+				)
+				(hide yes)
+			)
+		)
+		(property "Description" "Power symbol creates a global label with name \"GND\" , ground"
+			(at 106.68 132.08 0)
 			(effects
 				(font
@@
 		)
 		(instances
-			(project ""
+			(project "PSoM_nRF52840_00"
 				(path "/14b8af2e-80ef-48c8-890f-5f81b4faa854/a8f40f14-1954-4df1-a27b-4ef4decd9fbc"
-					(reference "SHIPHLD1")
+					(reference "#PWR011")
 					(unit 1)
 				)
@@
 	(symbol
 		(lib_id "Component_lib:R")
-		(at 91.44 116.84 0)
+		(at 83.82 116.84 0)
 		(unit 1)
 		(exclude_from_sim no)
@@
 		(fields_autoplaced yes)
 		(property "Reference" "R203"
-			(at 93.98 119.3799 0)
+			(at 86.36 119.3799 0)
 			(effects
 				(font
@@
 		)
 		(property "Value" "47k"
-			(at 93.98 121.9199 0)
+			(at 86.36 121.9199 0)
 			(effects
 				(font
@@
 		)
 		(property "Footprint" "Resistor_SMD:R_0201_0603Metric"
-			(at 89.662 120.65 90)
+			(at 82.042 120.65 90)
 			(effects
 				(font
@@
 		)
 		(property "Datasheet" "~"
-			(at 91.44 120.65 0)
+			(at 83.82 120.65 0)
 			(effects
 				(font
@@
 		)
 		(property "Description" "Resistor"
-			(at 91.44 116.84 0)
+			(at 83.82 116.84 0)
 			(effects
 				(font
@@
 	(symbol
 		(lib_id "Component_lib:R")
-		(at 101.6 116.84 0)
+		(at 93.98 116.84 0)
 		(unit 1)
 		(exclude_from_sim no)
@@
 		(fields_autoplaced yes)
 		(property "Reference" "R204"
-			(at 104.14 119.3799 0)
+			(at 96.52 119.3799 0)
 			(effects
 				(font
@@
 		)
 		(property "Value" "470k"
-			(at 104.14 121.9199 0)
+			(at 96.52 121.9199 0)
 			(effects
 				(font
@@
 		)
 		(property "Footprint" "Resistor_SMD:R_0201_0603Metric"
-			(at 99.822 120.65 90)
+			(at 92.202 120.65 90)
 			(effects
 				(font
@@
 		)
 		(property "Datasheet" "~"
-			(at 101.6 120.65 0)
+			(at 93.98 120.65 0)
 			(effects
 				(font
@@
 		)
 		(property "Description" "Resistor"
-			(at 101.6 116.84 0)
+			(at 93.98 116.84 0)
 			(effects
 				(font
@@
 		(lib_name "GND_1")
 		(lib_id "power:GND")
-		(at 91.44 127 0)
+		(at 83.82 127 0)
 		(unit 1)
 		(exclude_from_sim no)
@@
 		(fields_autoplaced yes)
 		(property "Reference" "#PWR010"
-			(at 91.44 133.35 0)
+			(at 83.82 133.35 0)
 			(effects
 				(font
@@
 		)
 		(property "Value" "GND"
-			(at 91.44 132.08 0)
+			(at 83.82 132.08 0)
 			(effects
 				(font
@@
 		)
 		(property "Footprint" ""
-			(at 91.44 127 0)
+			(at 83.82 127 0)
 			(effects
 				(font
@@
 		)
 		(property "Datasheet" ""
-			(at 91.44 127 0)
+			(at 83.82 127 0)
 			(effects
 				(font
@@
 		)
 		(property "Description" "Power symbol creates a global label with name \"GND\" , ground"
-			(at 91.44 127 0)
-			(effects
-				(font
+			(at 83.82 127 0)
+			(effects
+				(font
