File: Hardware/PSoM_ESP32_PICO_D4/PSoM_ESP32_PICO_D4_00/ESP32PICOD4.kicad_sch (KiCad schematic)
At the start: 15 parts, among them SW401 SW_Push, SW402 SW_Push, U401 ESP32-PICO-D4

Commit message: Final pinout for PSoM_ESP32_PICO_D4
Connections:
- no-connect marks 5 -> 6
Changed lines of the file:
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@@
 		(at 101.6 111.76)
+	)
+	(no_connect
+		(at 226.06 144.78)
 	)
 	(bus_entry
@@
 		)
 	)
+	(text_box "Only ADC1 is available\n(ADC2 used by wifi)"
+		(exclude_from_sim no)
+		(at 210.82 83.82 0)
+		(size 20.32 10.16)
+		(stroke
+			(width 0)
+			(type default)
+		)
+		(fill
+			(type none)
+		)
+		(effects
+			(font
+				(size 1.27 1.27)
+			)
+			(justify left top)
+		)
+	)

Commit message: First route for the PICO_D4
Added .gitignore
Modify at your own taste, this one will be tricky
Other:
- note added: "Internally PD Needs to be PD for boot Recommended as GPO -> Used for internal LED"
- note removed: "Internally PD Needs to be PD for boot Recommanded as GPO -> Used for internal LED"

Commit message: pico d4 routage terminé?
Parts:
- C401: footprint Capacitor_SMD:C_0201_0603Metric -> Capacitor_SMD:C_0603_1608Metric
- U401: footprint ESP32-PICO-D4_1 -> Component_lib:ESP32-PICO-D4_1
Changed lines of the file:
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@@
 			)
 		)
-		(property "Footprint" "ESP32-PICO-D4_1"
+		(property "Footprint" "Component_lib:ESP32-PICO-D4_1"
 			(at 113.03 50.165 0)
 			(effects
@@
 			)
 		)
-		(property "Footprint" "Capacitor_SMD:C_0201_0603Metric"
+		(property "Footprint" "Capacitor_SMD:C_0603_1608Metric"
 			(at 28.9052 83.82 0)
 			(effects
