File: Hardware/PSoM_Carrier/PSoM_Carrier_00/PSoM_Carrier_00.kicad_pcb (KiCad board)
At the start: 2 copper layers, 65.1 x 80 mm, 28 parts, among them J1 USB4510-03-1-A, J10 Conn_01x06, J11 Conn_01x04, J12 Conn_01x03, J13 Conn_01x02, J14 Conn_01x12, J15 Conn_01x03, J16 Conn_01x02, J17 Conn_01x06, J18 Conn_01x04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

Commit message: routing v0 is done
Parts:
- moved J10 89.1 mm to (100.7, 127.7), turned to 180 degrees
- moved J17 89.1 mm to (93.0, 127.7), turned to 180 degrees
- moved J1 87.0 mm to (143.8, 53.2), turned to 180 degrees
- moved J9 82.0 mm to (138.8, 127.7), turned to -90 degrees
- moved S2 80.1 mm to (112.3, 54.1), turned to 180 degrees
- moved S1 79.6 mm to (103.3, 54.1), turned to 180 degrees
- moved R2 78.6 mm to (147.4, 59.7)
- moved R1 75.6 mm to (139.8, 59.7), turned to 180 degrees
- moved J11 74.3 mm to (121.0, 127.7), turned to -90 degrees
- moved J7 68.7 mm to (137.2, 62.2)
- moved J20 68.5 mm to (138.8, 120.0), turned to -90 degrees
- moved J12 68.2 mm to (151.5, 74.3), turned to -90 degrees
- moved J15 65.9 mm to (151.5, 76.9), turned to -90 degrees
- moved J19 64.0 mm to (151.5, 79.4), turned to -90 degrees
- moved J22 60.9 mm to (120.8, 53.1), turned to 90 degrees
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Connections:
- J13 pad 1: /35 -> GND
- J13 pad 2: /37 -> /35
- J16 pad 2: GND -> /37
- J8 pad 1: /23 -> /52
- J8 pad 10: /46 -> /27
- J8 pad 11: /17 -> /25
- J8 pad 12: /52 -> /23
- J8 pad 2: /25 -> /17
- J8 pad 3: /27 -> /46
- J8 pad 4: /29 -> /32
- J8 pad 5: /31 -> /30
- J8 pad 6: /33 -> /39
- J8 pad 7: /39 -> /33
- J8 pad 8: /30 -> /31
- J8 pad 9: /32 -> /29
Routing:
- net /3V3: track 0.00 -> 205.5 mm, vias 0 -> 1
- net /36: track 0.00 -> 105.8 mm, vias 0 -> 2
- net /34: track 0.00 -> 98.9 mm, vias 0 -> 2
- net /VBUS: track 0.00 -> 97.1 mm, vias 0 -> 3
- net /19: track 0.00 -> 88.7 mm, vias 0 -> 1
- net /21: track 0.00 -> 83.1 mm, vias 0 -> 1
- net /48: track 0.00 -> 73.6 mm, vias 0 -> 1
- net /44: track 0.00 -> 67.6 mm, vias 0 -> 1
- net /50: track 0.00 -> 65.1 mm, vias 0 -> 1
- net /38: track 0.00 -> 65.0 mm, vias 0 -> 2
- net /42: track 0.00 -> 64.4 mm, vias 0 -> 1
- net /40: track 0.00 -> 60.0 mm, vias 0 -> 2
- net /17: track 0.00 -> 57.4 mm, vias 0 -> 1
- net /11: track 0.00 -> 51.5 mm
- net /23: track 0.00 -> 51.1 mm
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- added copper zone on B.Cu, net GND
- added copper zone on F.Cu, net GND
Other:
- board text added: "3V3"
- board text added: "MOSI MISO CLK CS"
- board text added: "PSoM_Carrier_00"
- board text added: "SPI1"
- board text added: "SPI2"
- board text added: "VBAT"
- board text added: "VBUS"
- board text added: "VSYS"

Commit message: updated routing
Parts:
- added G***: LOGO, Component_lib:puma_logo_14mm, F.Cu at (97.2, 59.3)
- moved J21 14.7 mm to (137.2, 127.0), turned to 180 degrees
- moved J18 11.4 mm to (111.9, 127.0), turned to 180 degrees
- moved J20 9.65 mm to (132.1, 127.0), turned to 180 degrees
- moved J9 4.19 mm to (134.6, 127.0), turned to 180 degrees
- moved J2 1.88 mm to (93.0, 83.8)
- moved J3 1.88 mm to (93.0, 78.7)
- moved J4 1.88 mm to (93.0, 73.7)
- moved J5 1.88 mm to (93.0, 68.6)
- moved J17 1.73 mm to (91.4, 127.0)
- moved J8 1.18 mm to (149.9, 94.0)
- moved J11 1.15 mm to (121.9, 127.0), turned to 180 degrees
- moved J14 1.15 mm to (152.4, 94.0)
- moved J10 1.15 mm to (101.6, 127.0)
- moved J13 1.15 mm to (152.4, 88.9)
- moved J16 1.15 mm to (152.4, 86.4)
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Routing:
- net /3V3: track 205.5 -> 189.6 mm
- net /48: track 73.6 -> 86.9 mm
- net /50: track 65.1 -> 75.6 mm
- net /13: track 49.8 -> 41.1 mm
- net /34: track 98.9 -> 107.5 mm
- net /15: track 48.4 -> 43.8 mm
- net /5: track 45.7 -> 41.3 mm
- net /19: track 88.7 -> 84.6 mm
- net /44: track 67.6 -> 71.6 mm
- net /36: track 105.8 -> 109.8 mm
- net /7: track 47.8 -> 44.0 mm
- net /37: track 31.1 -> 34.7 mm
- net /53: track 49.7 -> 46.7 mm
- net /RST: track 36.6 -> 39.4 mm
- net /32: track 44.4 -> 42.0 mm
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Other:
- board text added: "3V3 MOSI MISO CLK CS GND"
- board text added: "3V3 SDA SCL GND"
- board text added: "3V3 TX RX GND"
- board text added: "52 17 46 32 30 39 33 31 29 27 25 23"
- board text added: "ADC 3V3 GND"
- board text added: "ADC1 ADC2 ADC3"
- board text added: "DAC2 DAC1"
- board text added: "GND RST SWDCLK SDWIO 3V3"
- board text added: "I2C1"
- board text added: "I2C2"
- board text added: "UART 2 1 0"
- board text added: "VBUS D+ D- GND"
- board text removed: "MOSI MISO CLK CS"

Commit message: routing done, exported gerber file
Parts:
- added CS1-P43: TestPoint, TestPoint:TestPoint_Pad_1.0x1.0mm, F.Cu at (137.4, 95.6)
- added U1: W25Q128JVPIQ_TR, Component_lib:SON127P600X500X80-9N-D, F.Cu at (138.6, 88.0)
- moved G*** 16.7 mm to (112.0, 67.0)
- moved S1 1.12 mm to (103.5, 53.0)
- moved S2 1.12 mm to (112.5, 53.0)
Connections:
- S1 pad 2: GND -> /BOOT
- S1 pad 3: (no net) -> GND
- S1 pad 4: (no net) -> GND
- S2 pad 2: GND -> /RST
- S2 pad 3: (no net) -> GND
- S2 pad 4: (no net) -> GND
Routing:
- net /49: track 0.00 -> 23.2 mm, vias 0 -> 2
- net /43: track 0.00 -> 20.9 mm, vias 0 -> 2
- net /55: track 0.00 -> 18.3 mm, vias 0 -> 2
- net /53: track 46.7 -> 62.9 mm
- net /51: track 0.00 -> 15.9 mm, vias 0 -> 2
- net /57: track 0.00 -> 14.6 mm
- net /47: track 0.00 -> 14.2 mm
- net /45: track 0.00 -> 12.8 mm
- net GND: track 34.9 -> 44.2 mm, vias 2 -> 33
- net /RST: track 39.4 -> 43.8 mm
- net /5: track 41.3 -> 45.1 mm
- net /52: track 38.0 -> 41.7 mm
- net /BOOT: track 39.6 -> 43.2 mm
- net /46: track 47.9 -> 50.7 mm
- net /7: track 44.0 -> 46.7 mm
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Other:
- board size 65.1 x 80 mm -> 65 x 80 mm
- board text added: "BOOT"
- board text added: "RST"
