File: Hardware/PSoM_Carrier/PSoM_Carrier_00/PSoM_Carrier_00.kicad_sch (KiCad schematic)
At the start: 26 parts, among them J1 PSoM_ESP32S2_Carrier_Board, J10 Conn_01x03, J11 Conn_01x06, J12 Conn_01x06, J13 Conn_01x02, J14 Conn_01x02, J15 Conn_01x04, J16 Conn_01x04, J17 Conn_01x04, J18 Conn_01x04, J19 Conn_01x04, J2 USB4510-03-1-A, J20 Conn_01x04, J21 Conn_01x05, J3 53261-0371, J4 Conn_01x02, J5 Conn_01x02, J6 Conn_01x02, J7 Conn_01x03, J8 Conn_01x03, J9 Conn_01x02, SW1 450405020524

Commit message: finished schematic started layout
Parts:
- added J14, J8: Conn_01x12, Connector_PinHeader_2.54mm:PinHeader_1x12_P2.54mm_Vertical, symbol Connector_Generic:Conn_01x12
- J10: renamed from J11; footprint (none) -> Connector_PinHeader_2.54mm:PinHeader_1x06_P2.54mm_Vertical
- J11: renamed from J15; footprint (none) -> Connector_PinHeader_2.54mm:PinHeader_1x04_P2.54mm_Vertical
- J12: renamed from J7; footprint (none) -> Connector_PinHeader_2.54mm:PinHeader_1x03_P2.54mm_Vertical
- J13: footprint (none) -> Connector_PinHeader_2.54mm:PinHeader_1x02_P2.54mm_Vertical
- J15: renamed from J8; footprint (none) -> Connector_PinHeader_2.54mm:PinHeader_1x03_P2.54mm_Vertical
- J16: renamed from J14; footprint (none) -> Connector_PinHeader_2.54mm:PinHeader_1x02_P2.54mm_Vertical
- J17: renamed from J12; footprint (none) -> Connector_PinHeader_2.54mm:PinHeader_1x06_P2.54mm_Vertical
- J18: renamed from J16; footprint (none) -> Connector_PinHeader_2.54mm:PinHeader_1x04_P2.54mm_Vertical
- J19: renamed from J10; footprint (none) -> Connector_PinHeader_2.54mm:PinHeader_1x03_P2.54mm_Vertical
- J2: renamed from J9; footprint (none) -> Connector_PinHeader_2.54mm:PinHeader_1x02_P2.54mm_Vertical
- J20: renamed from J19; footprint (none) -> Connector_PinHeader_2.54mm:PinHeader_1x04_P2.54mm_Vertical
- J21: renamed from J20; footprint (none) -> Connector_PinHeader_2.54mm:PinHeader_1x04_P2.54mm_Vertical
- J22: renamed from J21; footprint (none) -> Connector_PinHeader_2.54mm:PinHeader_1x05_P2.54mm_Vertical
- J23: renamed from J1; footprint Component_lib:DF40C-60DS-0.4V(51) -> Component_lib:PSoM_ESP32S2_00
- J3: renamed from J4; footprint (none) -> Connector_PinHeader_2.54mm:PinHeader_1x02_P2.54mm_Vertical
- J4: renamed from J5; footprint (none) -> Connector_PinHeader_2.54mm:PinHeader_1x02_P2.54mm_Vertical
- J5: renamed from J6; footprint (none) -> Connector_PinHeader_2.54mm:PinHeader_1x02_P2.54mm_Vertical
- J7: renamed from J17; footprint (none) -> Connector_PinHeader_2.54mm:PinHeader_1x04_P2.54mm_Vertical
- J9: renamed from J18; footprint (none) -> Connector_PinHeader_2.54mm:PinHeader_1x04_P2.54mm_Vertical
- R1, R2: footprint (none) -> Resistor_SMD:R_0402_1005Metric
- renumbered J2 to J1, J3 to J6
Connections:
- net 11: now also J10.2 (Pin_2); no longer J10.5 (Pin_5)
- net 13: now also J11.3 (Pin_3); no longer J11.2 (Pin_2)
- net 15: now also J11.2 (Pin_2); no longer J11.3 (Pin_3)
- net 17: now also J12.3 (Pin_3), J8.11 (Pin_11); no longer J12.1 (Pin_1)
- net 19: now also J15.3 (Pin_3), J9.3 (Pin_3); no longer J12.2 (Pin_2), J9.2 (Pin_2)
- net 21: now also J19.3 (Pin_3), J9.2 (Pin_2); no longer J12.3 (Pin_3), J9.3 (Pin_3)
- net 23: now also J8.1 (Pin_1)
- net 25: now also J8.2 (Pin_2)
- net 27: now also J8.3 (Pin_3)
- net 29: now also J8.4 (Pin_4)
- net 30: now also J8.8 (Pin_8)
- net 31: now also J8.5 (Pin_5)
- net 32: now also J8.9 (Pin_9)
- net 33: now also J8.6 (Pin_6)
- net 34: now also J17.5 (Pin_5), J20.3 (Pin_3); no longer J17.2 (Pin_2), J20.2 (Pin_2)
- net 36: now also J17.4 (Pin_4), J20.2 (Pin_2); no longer J17.3 (Pin_3), J20.3 (Pin_3)
- net 38: now also J17.3 (Pin_3); no longer J17.4 (Pin_4)
- net 39: now also J8.7 (Pin_7)
- net 3V3: now also J10.6 (Pin_6), J11.4 (Pin_4), J12.2 (Pin_2), J17.6 (Pin_6), J18.4 (Pin_4), J19.2 (Pin_2), J20.4 (Pin_4), J21.4 (Pin_4), J22.5 (Pin_5), J5.2 (Pin_2), J9.4 (Pin_4); no longer J10.1 (Pin_1), J11.1 (Pin_1), J15.1 (Pin_1), J15.3 (Pin_3), J17.1 (Pin_1), J18.1 (Pin_1), J20.1 (Pin_1), J21.1 (Pin_1), J22.1 (Pin_1), J5.1 (Pin_1), J9.1 (Pin_1)
- net 40: now also J17.2 (Pin_2); no longer J17.5 (Pin_5)
- net 42: now also J18.3 (Pin_3); no longer J18.2 (Pin_2)
- net 44: now also J18.2 (Pin_2); no longer J18.3 (Pin_3)
- net 46: now also J8.10 (Pin_10)
- net 48: now also J21.2 (Pin_2); no longer J21.3 (Pin_3)
- net 5: now also J10.5 (Pin_5); no longer J10.2 (Pin_2)
- net 50: now also J21.3 (Pin_3), J22.4 (Pin_4); no longer J21.2 (Pin_2), J22.2 (Pin_2)
- net 52: now also J8.12 (Pin_12)
- net 53: now also J10.3 (Pin_3); no longer J10.4 (Pin_4)
- net 7: now also J10.4 (Pin_4); no longer J10.3 (Pin_3)
- net GND: now also J10.1 (Pin_1), J11.1 (Pin_1), J12.1 (Pin_1), J15.1 (Pin_1), J17.1 (Pin_1), J18.1 (Pin_1), J2.1 (Pin_1), J20.1 (Pin_1), J21.1 (Pin_1), J22.1 (Pin_1), J3.1 (Pin_1), J4.1 (Pin_1), J5.1 (Pin_1), J9.1 (Pin_1), J14.1 (Pin_1), J14.10 (Pin_10), J14.11 (Pin_11), J14.12 (Pin_12), J14.2 (Pin_2), J14.3 (Pin_3), J14.4 (Pin_4), J14.5 (Pin_5), J14.6 (Pin_6), J14.7 (Pin_7), J14.8 (Pin_8), J14.9 (Pin_9); no longer J10.6 (Pin_6), J11.4 (Pin_4), J17.6 (Pin_6), J18.4 (Pin_4), J19.2 (Pin_2), J19.3 (Pin_3), J2.2 (Pin_2), J20.4 (Pin_4), J21.4 (Pin_4), J22.5 (Pin_5), J3.2 (Pin_2), J4.2 (Pin_2), J5.2 (Pin_2), J9.4 (Pin_4)
- net RST: now also J22.2 (Pin_2); no longer J22.4 (Pin_4)
- net VBAT_SWITCHED: now also J2.2 (Pin_2); no longer J2.1 (Pin_1)
- net VBUS: now also J3.2 (Pin_2); no longer J3.1 (Pin_1)
- net VSYS: now also J4.2 (Pin_2); no longer J4.1 (Pin_1)
Other:
- note added: "GPIO"
- moved on the sheet: J12, J13, J15, J16, J19, J2, J20, J21, J22, J23, J3, J4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

Commit message: routing v0 is done
Connections:
- net 17: now also J8.2 (Pin_2); no longer J8.11 (Pin_11)
- net 23: now also J8.12 (Pin_12); no longer J8.1 (Pin_1)
- net 25: now also J8.11 (Pin_11); no longer J8.2 (Pin_2)
- net 27: now also J8.10 (Pin_10); no longer J8.3 (Pin_3)
- net 29: now also J8.9 (Pin_9); no longer J8.4 (Pin_4)
- net 30: now also J8.5 (Pin_5); no longer J8.8 (Pin_8)
- net 31: now also J8.8 (Pin_8); no longer J8.5 (Pin_5)
- net 32: now also J8.4 (Pin_4); no longer J8.9 (Pin_9)
- net 33: now also J8.7 (Pin_7); no longer J8.6 (Pin_6)
- net 35: now also J13.2 (Pin_2); no longer J13.1 (Pin_1)
- net 37: now also J16.2 (Pin_2); no longer J13.2 (Pin_2)
- net 39: now also J8.6 (Pin_6); no longer J8.7 (Pin_7)
- net 46: now also J8.3 (Pin_3); no longer J8.10 (Pin_10)
- net 52: now also J8.1 (Pin_1); no longer J8.12 (Pin_12)
- net GND: now also J13.1 (Pin_1); no longer J16.2 (Pin_2)
Other:
- moved on the sheet: J16
Changed lines of the file:
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@@
 	)
 	(junction
-		(at 132.08 187.96)
-		(diameter 0)
-		(color 0 0 0 0)
-	)
-	(junction
 		(at 43.18 40.64)
 		(diameter 0)
@@
 	(wire
 		(pts
-			(xy 132.08 187.96) (xy 134.62 187.96)
-		)
-		(stroke
-			(width 0)
-			(type default)
-		)
-	)
-	(wire
-		(pts
 			(xy 60.96 43.18) (xy 60.96 45.72)
 		)
@@
 	(wire
 		(pts
-			(xy 109.22 187.96) (xy 106.68 187.96)
-		)
-		(stroke
-			(width 0)
-			(type default)
-		)
-	)
-	(wire
-		(pts
 			(xy 142.24 25.4) (xy 144.78 25.4)
 		)
@@
 	(wire
 		(pts
+			(xy 109.22 187.96) (xy 106.68 187.96)
+		)
+		(stroke
+			(width 0)
+			(type default)
+		)
+	)
+	(wire
+		(pts
 			(xy 137.16 88.9) (xy 139.7 88.9)
 		)
@@
 	(wire
 		(pts
+			(xy 106.68 185.42) (xy 109.22 185.42)
+		)
+		(stroke
+			(width 0)
+			(type default)
+		)
+	)
+	(wire
+		(pts
 			(xy 121.92 162.56) (xy 124.46 162.56)
 		)
@@
 	(wire
 		(pts
-			(xy 109.22 185.42) (xy 106.68 185.42)
-		)
-		(stroke
-			(width 0)
-			(type default)
-		)
-	)
-	(wire
-		(pts
 			(xy 246.38 93.98) (xy 251.46 93.98)
 		)
@@
 	(wire
 		(pts
-			(xy 132.08 190.5) (xy 132.08 187.96)
+			(xy 137.16 187.96) (xy 137.16 190.5)
 		)
 		(stroke
@@
 	(wire
 		(pts
-			(xy 132.08 187.96) (xy 132.08 185.42)
+			(xy 246.38 149.86) (xy 251.46 149.86)
 		)
 		(stroke
@@
 	(wire
 		(pts
-			(xy 246.38 149.86) (xy 251.46 149.86)
+			(xy 137.16 185.42) (xy 139.7 185.42)
 		)
 		(stroke
@@
 	(wire
 		(pts
-			(xy 132.08 185.42) (xy 134.62 185.42)
+			(xy 137.16 187.96) (xy 139.7 187.96)
 		)
 		(stroke
@@
 	(wire
 		(pts
+			(xy 106.68 187.96) (xy 106.68 190.5)
+		)
+		(stroke
+			(width 0)
+			(type default)
+		)
+	)
+	(wire
+		(pts
 			(xy 116.84 121.92) (xy 119.38 121.92)
 		)
@@
 	)
 	(label "32"
-		(at 101.6 132.08 180)
+		(at 101.6 119.38 180)
 		(effects
 			(font
@@
 	)
 	(label "52"
-		(at 101.6 139.7 180)
+		(at 101.6 111.76 180)
 		(effects
 			(font
@@
 	)
 	(label "29"
-		(at 101.6 119.38 180)
+		(at 101.6 132.08 180)
 		(effects
 			(font
@@
 	)
 	(label "46"
-		(at 101.6 134.62 180)
+		(at 101.6 116.84 180)
 		(effects
 			(font
@@
 	)
 	(label "33"
-		(at 101.6 124.46 180)
+		(at 101.6 127 180)
 		(effects
 			(font
@@
 	)
 	(label "31"
-		(at 101.6 121.92 180)
+		(at 101.6 129.54 180)
 		(effects
 			(font
@@
 	)
 	(label "25"
-		(at 101.6 114.3 180)
+		(at 101.6 137.16 180)
 		(effects
 			(font
@@
 	)
 	(label "27"
-		(at 101.6 116.84 180)
+		(at 101.6 134.62 180)
 		(effects
 			(font
@@
 	)
 	(label "17"
-		(at 101.6 137.16 180)
+		(at 101.6 114.3 180)
 		(effects
 			(font
@@
 	)
 	(label "23"
-		(at 101.6 111.76 180)
+		(at 101.6 139.7 180)
 		(effects
 			(font
@@
 	)
 	(label "39"
-		(at 101.6 127 180)
+		(at 101.6 124.46 180)
 		(effects
 			(font
@@
 	)
 	(label "DAC2"
-		(at 106.68 187.96 180)
+		(at 137.16 185.42 180)
 		(effects
 			(font
@@
 	)
 	(label "30"
-		(at 101.6 129.54 180)
+		(at 101.6 121.92 180)
 		(effects
 			(font
@@
 	(symbol
 		(lib_id "power:GND")
+		(at 106.68 190.5 0)
+		(unit 1)
+		(exclude_from_sim no)
+		(in_bom yes)
+		(on_board yes)
+		(dnp no)
+		(fields_autoplaced yes)
+		(property "Reference" "#PWR029"
+			(at 106.68 196.85 0)
+			(effects
+				(font
+					(size 1.27 1.27)
+				)
+				(hide yes)
+			)
+		)
+		(property "Value" "GND"
+			(at 106.68 195.58 0)
+			(effects
+				(font
+					(size 1.27 1.27)
+				)
+			)
+		)
+		(property "Footprint" ""
+			(at 106.68 190.5 0)
+			(effects
+				(font
+					(size 1.27 1.27)
+				)
+				(hide yes)
+			)
+		)
+		(property "Datasheet" ""
+			(at 106.68 190.5 0)
+			(effects
+				(font
+					(size 1.27 1.27)
+				)
+				(hide yes)
+			)
+		)
+		(property "Description" "Power symbol creates a global label with name \"GND\" , ground"
+			(at 106.68 190.5 0)
+			(effects
+				(font
+					(size 1.27 1.27)
+				)
+				(hide yes)
+			)
+		)
+		(pin "1"
+		)
+		(instances
+			(project "PSoM_Carrier_00"
+				(path "/de611377-129e-43ca-975d-e8727f221d2e"
+					(reference "#PWR029")
+					(unit 1)
+				)
+			)
+		)
+	)
+	(symbol
+		(lib_id "power:GND")
 		(at 142.24 33.02 0)
 		(unit 1)
@@
 	(symbol
 		(lib_id "power:GND")
-		(at 132.08 190.5 0)
+		(at 137.16 190.5 0)
 		(unit 1)
 		(exclude_from_sim no)
@@
 		(fields_autoplaced yes)
 		(property "Reference" "#PWR016"
-			(at 132.08 196.85 0)
+			(at 137.16 196.85 0)
 			(effects
 				(font
@@
 		)
 		(property "Value" "GND"
-			(at 132.08 195.58 0)
+			(at 137.16 195.58 0)
 			(effects
 				(font
@@
 		)
 		(property "Footprint" ""
-			(at 132.08 190.5 0)
+			(at 137.16 190.5 0)
 			(effects
 				(font
@@
 		)
 		(property "Datasheet" ""
-			(at 132.08 190.5 0)
+			(at 137.16 190.5 0)
 			(effects
 				(font
@@
 		)
 		(property "Description" "Power symbol creates a global label with name \"GND\" , ground"
-			(at 132.08 190.5 0)
+			(at 137.16 190.5 0)
 			(effects
 				(font
@@
 	(symbol
 		(lib_id "Connector_Generic:Conn_01x02")
-		(at 114.3 185.42 0)
+		(at 114.3 187.96 0)
+		(mirror x)
 		(unit 1)
 		(exclude_from_sim no)
@@
 		(on_board yes)
 		(dnp no)
-		(fields_autoplaced yes)
 		(property "Reference" "J13"
-			(at 116.84 185.4199 0)
+			(at 116.84 187.9601 0)
 			(effects
 				(font
@@
 		)
 		(property "Value" "Conn_01x02"
-			(at 116.84 187.9599 0)
+			(at 116.84 185.4201 0)
 			(effects
 				(font
@@
 		)
 		(property "Footprint" "Connector_PinHeader_2.54mm:PinHeader_1x02_P2.54mm_Vertical"
-			(at 114.3 185.42 0)
+			(at 114.3 187.96 0)
 			(effects
 				(font
@@
 		)
 		(property "Datasheet" "~"
-			(at 114.3 185.42 0)
+			(at 114.3 187.96 0)
 			(effects
 				(font
@@
 		)
 		(property "Description" "Generic connector, single row, 01x02, script generated (kicad-library-utils/schlib/autogen/connector/)"
-			(at 114.3 185.42 0)
+			(at 114.3 187.96 0)
 			(effects
 				(font
@@
 	(symbol
 		(lib_id "Connector_Generic:Conn_01x02")
-		(at 139.7 185.42 0)
+		(at 144.78 187.96 0)
+		(mirror x)
 		(unit 1)
 		(exclude_from_sim no)
@@
 		(on_board yes)
 		(dnp no)
-		(fields_autoplaced yes)
 		(property "Reference" "J16"
-			(at 142.24 185.4199 0)
+			(at 147.32 187.9601 0)
 			(effects
 				(font
@@
 		)
 		(property "Value" "Conn_01x02"
-			(at 142.24 187.9599 0)
+			(at 147.32 185.4201 0)
 			(effects
 				(font
@@
 		)
 		(property "Footprint" "Connector_PinHeader_2.54mm:PinHeader_1x02_P2.54mm_Vertical"
-			(at 139.7 185.42 0)
+			(at 144.78 187.96 0)
 			(effects
 				(font
@@
 		)
 		(property "Datasheet" "~"
-			(at 139.7 185.42 0)
+			(at 144.78 187.96 0)
 			(effects
 				(font
@@
 		)
 		(property "Description" "Generic connector, single row, 01x02, script generated (kicad-library-utils/schlib/autogen/connector/)"
-			(at 139.7 185.42 0)
+			(at 144.78 187.96 0)
 			(effects
 				(font

Commit message: routing done, exported gerber file
Parts:
- added TP1: TestPoint, TestPoint:TestPoint_Pad_1.0x1.0mm, symbol Connector:TestPoint
- added U1: W25Q128JVPIQ_TR, Component_lib:SON127P600X500X80-9N-D, symbol Component_lib:W25Q128JVPIQ
Connections:
- net 43: now also TP1.1
- net 45: now also U1.8 (VCC)
- net 47: now also U1.7 (~{HOLD_OR_RESET_(IO3)})
- net 49: now also U1.3 (~{WP_(IO2)})
- net 51: now also U1.1 (~{CS})
- net 53: now also U1.6 (CLK)
- net 55: now also U1.2 (DO_(IO1))
- net 57: now also U1.5 (DI_(IO0))
- net BOOT: now also S1.2 (1)
- net GND: now also S1.3 (2), S1.4 (2), S2.3 (2), S2.4 (2), U1.4 (GND), U1.9 (EP); no longer S1.2, S2.2
- net RST: now also S2.2 (1)
Other:
- moved on the sheet: J10, J11, J12, J13, J14, J15, J16, J17, J18, J19, J20, J21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
